File: MMS3/MCU.kicad_sch (KiCad schematic)
At the start: 39 parts, among them SW3 TC-6615Z-12.5-260, SW5 TC-6615Z-12.5-260, U1 STM32F405RGTx, X1 X32258MOB4SI, X2 Q13FC1350000400

Commit message: finished routing
Other:
- title: MMS3 -> MMS3 MCU ESP32-C6
