File: MMS3/CAN_TR.kicad_sch (KiCad schematic)
At the start: 6 parts, among them U500 TJA1044GTK_3Z

Commit message: finished routing
Parts:
- C5: DNP_Basic (none) -> DNP; Manufacturer Samsung Electro-Mechanics -> (none)
- C6: renamed from C3; DNP_Basic (none) -> DNP; Manufacturer Samsung Electro-Mechanics -> (none)
- R9: renamed from R500; DNP_Basic (none) -> DNP; Manufacturer UNI-ROYAL(Uniroyal Elec) -> (none)
- TP1: DNP_Basic (none) -> DNP
- TP2: renamed from TP3; DNP_Basic (none) -> DNP
- U1: renamed from U500; DNP_Basic (none) -> DNP
Other:
- title: MMS3 -> MMS3 MCU ESP32-C6

Commit message: temp commit
Parts:
- renumbered C5 to C3, C6 to C4, R9 to R7
Changed lines of the file:
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@@
 		(in_pos_files yes)
 		(dnp no)
-		(property "Reference" "R9"
+		(property "Reference" "R7"
 			(at 180.34 113.03 0)
 			(show_name no)
@@
 		(instances
 			(project "MMS3_ESP32-C6"
-				(path "/712cea22-140d-4c92-923f-f4998caf3ecd/113a3eca-1aef-4188-a06d-d5e25149d583"
-					(reference "R11")
-					(unit 1)
-				)
-				(path "/712cea22-140d-4c92-923f-f4998caf3ecd/9f611e2f-54d9-422f-9f20-2d94caaac009"
-					(reference "R9")
+				(path "/712cea22-140d-4c92-923f-f4998caf3ecd/0aa97c32-fb04-42d1-b504-a6b2d0473b51"
+					(reference "R12")
+					(unit 1)
+				)
+				(path "/712cea22-140d-4c92-923f-f4998caf3ecd/599e2418-6476-4380-932e-471cd9f203c3"
+					(reference "R7")
 					(unit 1)
 				)
@@
 		(dnp no)
 		(fields_autoplaced yes)
-		(property "Reference" "C6"
+		(property "Reference" "C4"
 			(at 194.31 77.47 90)
 			(show_name no)
@@
 		(instances
 			(project "MMS3_ESP32-C6"
-				(path "/712cea22-140d-4c92-923f-f4998caf3ecd/113a3eca-1aef-4188-a06d-d5e25149d583"
-					(reference "C8")
-					(unit 1)
-				)
-				(path "/712cea22-140d-4c92-923f-f4998caf3ecd/9f611e2f-54d9-422f-9f20-2d94caaac009"
-					(reference "C6")
+				(path "/712cea22-140d-4c92-923f-f4998caf3ecd/0aa97c32-fb04-42d1-b504-a6b2d0473b51"
+					(reference "C7")
+					(unit 1)
+				)
+				(path "/712cea22-140d-4c92-923f-f4998caf3ecd/599e2418-6476-4380-932e-471cd9f203c3"
+					(reference "C4")
 					(unit 1)
 				)
@@
 		(instances
 			(project "MMS3_ESP32-C6"
-				(path "/712cea22-140d-4c92-923f-f4998caf3ecd/113a3eca-1aef-4188-a06d-d5e25149d583"
+				(path "/712cea22-140d-4c92-923f-f4998caf3ecd/0aa97c32-fb04-42d1-b504-a6b2d0473b51"
 					(reference "#PWR0517")
 					(unit 1)
 				)
-				(path "/712cea22-140d-4c92-923f-f4998caf3ecd/9f611e2f-54d9-422f-9f20-2d94caaac009"
+				(path "/712cea22-140d-4c92-923f-f4998caf3ecd/599e2418-6476-4380-932e-471cd9f203c3"
 					(reference "#PWR0511")
 					(unit 1)
@@
 		(instances
 			(project "MMS3_ESP32-C6"
-				(path "/712cea22-140d-4c92-923f-f4998caf3ecd/113a3eca-1aef-4188-a06d-d5e25149d583"
+				(path "/712cea22-140d-4c92-923f-f4998caf3ecd/0aa97c32-fb04-42d1-b504-a6b2d0473b51"
 					(reference "TP4")
 					(unit 1)
 				)
-				(path "/712cea22-140d-4c92-923f-f4998caf3ecd/9f611e2f-54d9-422f-9f20-2d94caaac009"
+				(path "/712cea22-140d-4c92-923f-f4998caf3ecd/599e2418-6476-4380-932e-471cd9f203c3"
 					(reference "TP2")
 					(unit 1)
@@
 		(dnp no)
 		(fields_autoplaced yes)
-		(property "Reference" "C5"
+		(property "Reference" "C3"
 			(at 137.16 76.2 90)
 			(show_name no)
@@
 		(instances
 			(project "MMS3_ESP32-C6"
-				(path "/712cea22-140d-4c92-923f-f4998caf3ecd/113a3eca-1aef-4188-a06d-d5e25149d583"
-					(reference "C7")
-					(unit 1)
-				)
-				(path "/712cea22-140d-4c92-923f-f4998caf3ecd/9f611e2f-54d9-422f-9f20-2d94caaac009"
-					(reference "C5")
+				(path "/712cea22-140d-4c92-923f-f4998caf3ecd/0aa97c32-fb04-42d1-b504-a6b2d0473b51"
+					(reference "C6")
+					(unit 1)
+				)
+				(path "/712cea22-140d-4c92-923f-f4998caf3ecd/599e2418-6476-4380-932e-471cd9f203c3"
+					(reference "C3")
 					(unit 1)
 				)
@@
 		(instances
 			(project "MMS3_ESP32-C6"
-				(path "/712cea22-140d-4c92-923f-f4998caf3ecd/113a3eca-1aef-4188-a06d-d5e25149d583"
-					(reference "U7")
-					(unit 1)
-				)
-				(path "/712cea22-140d-4c92-923f-f4998caf3ecd/9f611e2f-54d9-422f-9f20-2d94caaac009"
+				(path "/712cea22-140d-4c92-923f-f4998caf3ecd/0aa97c32-fb04-42d1-b504-a6b2d0473b51"
+					(reference "U6")
+					(unit 1)
+				)
+				(path "/712cea22-140d-4c92-923f-f4998caf3ecd/599e2418-6476-4380-932e-471cd9f203c3"
 					(reference "U1")
 					(unit 1)
@@
 		(instances
 			(project "MMS3_ESP32-C6"
-				(path "/712cea22-140d-4c92-923f-f4998caf3ecd/113a3eca-1aef-4188-a06d-d5e25149d583"
+				(path "/712cea22-140d-4c92-923f-f4998caf3ecd/0aa97c32-fb04-42d1-b504-a6b2d0473b51"
 					(reference "#PWR0514")
 					(unit 1)
 				)
-				(path "/712cea22-140d-4c92-923f-f4998caf3ecd/9f611e2f-54d9-422f-9f20-2d94caaac009"
+				(path "/712cea22-140d-4c92-923f-f4998caf3ecd/599e2418-6476-4380-932e-471cd9f203c3"
 					(reference "#PWR0508")
 					(unit 1)
@@
 		(instances
 			(project "MMS3_ESP32-C6"
-				(path "/712cea22-140d-4c92-923f-f4998caf3ecd/113a3eca-1aef-4188-a06d-d5e25149d583"
+				(path "/712cea22-140d-4c92-923f-f4998caf3ecd/0aa97c32-fb04-42d1-b504-a6b2d0473b51"
 					(reference "TP3")
 					(unit 1)
 				)
-				(path "/712cea22-140d-4c92-923f-f4998caf3ecd/9f611e2f-54d9-422f-9f20-2d94caaac009"
+				(path "/712cea22-140d-4c92-923f-f4998caf3ecd/599e2418-6476-4380-932e-471cd9f203c3"
 					(reference "TP1")
 					(unit 1)
@@
 		(instances
 			(project "MMS3_ESP32-C6"
-				(path "/712cea22-140d-4c92-923f-f4998caf3ecd/113a3eca-1aef-4188-a06d-d5e25149d583"
+				(path "/712cea22-140d-4c92-923f-f4998caf3ecd/0aa97c32-fb04-42d1-b504-a6b2d0473b51"
 					(reference "#PWR0515")
 					(unit 1)
 				)
-				(path "/712cea22-140d-4c92-923f-f4998caf3ecd/9f611e2f-54d9-422f-9f20-2d94caaac009"
+				(path "/712cea22-140d-4c92-923f-f4998caf3ecd/599e2418-6476-4380-932e-471cd9f203c3"
 					(reference "#PWR0510")
 					(unit 1)
@@
 		(instances
 			(project "MMS3_ESP32-C6"
-				(path "/712cea22-140d-4c92-923f-f4998caf3ecd/113a3eca-1aef-4188-a06d-d5e25149d583"
+				(path "/712cea22-140d-4c92-923f-f4998caf3ecd/0aa97c32-fb04-42d1-b504-a6b2d0473b51"
 					(reference "#PWR0516")
 					(unit 1)
 				)
-				(path "/712cea22-140d-4c92-923f-f4998caf3ecd/9f611e2f-54d9-422f-9f20-2d94caaac009"
+				(path "/712cea22-140d-4c92-923f-f4998caf3ecd/599e2418-6476-4380-932e-471cd9f203c3"
 					(reference "#PWR0509")
 					(unit 1)
@@
 		(instances
 			(project "MMS3_ESP32-C6"
-				(path "/712cea22-140d-4c92-923f-f4998caf3ecd/113a3eca-1aef-4188-a06d-d5e25149d583"
+				(path "/712cea22-140d-4c92-923f-f4998caf3ecd/0aa97c32-fb04-42d1-b504-a6b2d0473b51"
 					(reference "#PWR0513")
 					(unit 1)
 				)
-				(path "/712cea22-140d-4c92-923f-f4998caf3ecd/9f611e2f-54d9-422f-9f20-2d94caaac009"
+				(path "/712cea22-140d-4c92-923f-f4998caf3ecd/599e2418-6476-4380-932e-471cd9f203c3"
 					(reference "#PWR0507")
 					(unit 1)
@@
 		(instances
 			(project "MMS3_ESP32-C6"
-				(path "/712cea22-140d-4c92-923f-f4998caf3ecd/113a3eca-1aef-4188-a06d-d5e25149d583"
+				(path "/712cea22-140d-4c92-923f-f4998caf3ecd/0aa97c32-fb04-42d1-b504-a6b2d0473b51"
 					(reference "#PWR0512")
 					(unit 1)
 				)
-				(path "/712cea22-140d-4c92-923f-f4998caf3ecd/9f611e2f-54d9-422f-9f20-2d94caaac009"
+				(path "/712cea22-140d-4c92-923f-f4998caf3ecd/599e2418-6476-4380-932e-471cd9f203c3"
 					(reference "#PWR0506")
 					(unit 1)

Commit message: eem, done?
Parts:
- TP1, TP2: now not fitted; now left out of the parts list
