File: MMS3/I2C_Flash.kicad_sch (KiCad schematic)
At the start: 9 parts, among them U6 AT24C256C

Commit message: finished routing
Parts:
- removed C27: 100nF, PCM_JLCPCB:C_0402, symbol PCM_JLCPCB-Capacitors:0402,100nF,(2)
- removed R23, R24, R25, R26, R28, R29, R30: 10kΩ, PCM_JLCPCB:R_0402, symbol PCM_JLCPCB-Resistors:0402,10kΩ
- added C11: 100nF, PCM_JLCPCB:C_0603, symbol PCM_JLCPCB-Capacitors:0603,100nF
- added R16, R17, R18, R19, R20, R21, R22: 10kΩ, PCM_JLCPCB:R_0603, symbol PCM_JLCPCB-Resistors:0603,10kΩ
- U6: Manufacturer Microchip Tech -> (none)
Connections:
- net +3V3: now also C11.1, R17.1, R18.1, R19.1
- net A1: now also R18.2, R21.1
- net A2: now also R17.2, R22.1
- net GND: now also C11.2, R16.2, R20.2, R21.2, R22.2
- net I2C_Memory_addr: now also R19.2, R20.1
- net at U6.7 (WP): now also R16.1
Other:
- title: MMS3 -> MMS3 MCU ESP32-C6

Commit message: temp commit
Parts:
- renumbered C11 to C16, R16 to R30, R17 to R31, R22 to R32, R18 to R35, R21 to R40, R19 to R41, R20 to R42, U6 to U10
Changed lines of the file:
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@@
 		(instances
 			(project "MMS3_ESP32-C6"
-				(path "/712cea22-140d-4c92-923f-f4998caf3ecd/c085740e-6122-4df8-b6d1-901cece69bb5"
+				(path "/712cea22-140d-4c92-923f-f4998caf3ecd/252530b9-e462-46c8-9362-2c7b584836c4"
 					(reference "#PWR037")
 					(unit 1)
@@
 		(instances
 			(project "MMS3_ESP32-C6"
-				(path "/712cea22-140d-4c92-923f-f4998caf3ecd/c085740e-6122-4df8-b6d1-901cece69bb5"
+				(path "/712cea22-140d-4c92-923f-f4998caf3ecd/252530b9-e462-46c8-9362-2c7b584836c4"
 					(reference "#PWR042")
 					(unit 1)
@@
 		(dnp no)
 		(fields_autoplaced yes)
-		(property "Reference" "C11"
+		(property "Reference" "C16"
 			(at 73.66 95.2499 0)
 			(show_name no)
@@
 		(instances
 			(project "MMS3_ESP32-C6"
-				(path "/712cea22-140d-4c92-923f-f4998caf3ecd/c085740e-6122-4df8-b6d1-901cece69bb5"
-					(reference "C11")
+				(path "/712cea22-140d-4c92-923f-f4998caf3ecd/252530b9-e462-46c8-9362-2c7b584836c4"
+					(reference "C16")
 					(unit 1)
 				)
@@
 		(dnp no)
 		(fields_autoplaced yes)
-		(property "Reference" "R19"
+		(property "Reference" "R41"
 			(at 182.88 87.6299 0)
 			(show_name no)
@@
 		(instances
 			(project "MMS3_ESP32-C6"
-				(path "/712cea22-140d-4c92-923f-f4998caf3ecd/c085740e-6122-4df8-b6d1-901cece69bb5"
-					(reference "R19")
+				(path "/712cea22-140d-4c92-923f-f4998caf3ecd/252530b9-e462-46c8-9362-2c7b584836c4"
+					(reference "R41")
 					(unit 1)
 				)
@@
 		(instances
 			(project "MMS3_ESP32-C6"
-				(path "/712cea22-140d-4c92-923f-f4998caf3ecd/c085740e-6122-4df8-b6d1-901cece69bb5"
+				(path "/712cea22-140d-4c92-923f-f4998caf3ecd/252530b9-e462-46c8-9362-2c7b584836c4"
 					(reference "#PWR041")
 					(unit 1)
@@
 		(dnp yes)
 		(fields_autoplaced yes)
-		(property "Reference" "R21"
+		(property "Reference" "R40"
 			(at 175.26 105.4099 0)
 			(show_name no)
@@
 		(instances
 			(project "MMS3_ESP32-C6"
-				(path "/712cea22-140d-4c92-923f-f4998caf3ecd/c085740e-6122-4df8-b6d1-901cece69bb5"
-					(reference "R21")
+				(path "/712cea22-140d-4c92-923f-f4998caf3ecd/252530b9-e462-46c8-9362-2c7b584836c4"
+					(reference "R40")
 					(unit 1)
 				)
@@
 		(instances
 			(project "MMS3_ESP32-C6"
-				(path "/712cea22-140d-4c92-923f-f4998caf3ecd/c085740e-6122-4df8-b6d1-901cece69bb5"
+				(path "/712cea22-140d-4c92-923f-f4998caf3ecd/252530b9-e462-46c8-9362-2c7b584836c4"
 					(reference "#PWR044")
 					(unit 1)
@@
 		(dnp no)
 		(fields_autoplaced yes)
-		(property "Reference" "R18"
+		(property "Reference" "R35"
 			(at 175.26 87.6299 0)
 			(show_name no)
@@
 		(instances
 			(project "MMS3_ESP32-C6"
-				(path "/712cea22-140d-4c92-923f-f4998caf3ecd/c085740e-6122-4df8-b6d1-901cece69bb5"
-					(reference "R18")
+				(path "/712cea22-140d-4c92-923f-f4998caf3ecd/252530b9-e462-46c8-9362-2c7b584836c4"
+					(reference "R35")
 					(unit 1)
 				)
@@
 		(dnp no)
 		(fields_autoplaced yes)
-		(property "Reference" "R17"
+		(property "Reference" "R31"
 			(at 167.64 87.6299 0)
 			(show_name no)
@@
 		(instances
 			(project "MMS3_ESP32-C6"
-				(path "/712cea22-140d-4c92-923f-f4998caf3ecd/c085740e-6122-4df8-b6d1-901cece69bb5"
-					(reference "R17")
+				(path "/712cea22-140d-4c92-923f-f4998caf3ecd/252530b9-e462-46c8-9362-2c7b584836c4"
+					(reference "R31")
 					(unit 1)
 				)
@@
 		(instances
 			(project "MMS3_ESP32-C6"
-				(path "/712cea22-140d-4c92-923f-f4998caf3ecd/c085740e-6122-4df8-b6d1-901cece69bb5"
+				(path "/712cea22-140d-4c92-923f-f4998caf3ecd/252530b9-e462-46c8-9362-2c7b584836c4"
 					(reference "#PWR040")
 					(unit 1)
@@
 		(dnp yes)
 		(fields_autoplaced yes)
-		(property "Reference" "R20"
+		(property "Reference" "R42"
 			(at 182.88 105.4099 0)
 			(show_name no)
@@
 		(instances
 			(project "MMS3_ESP32-C6"
-				(path "/712cea22-140d-4c92-923f-f4998caf3ecd/c085740e-6122-4df8-b6d1-901cece69bb5"
-					(reference "R20")
+				(path "/712cea22-140d-4c92-923f-f4998caf3ecd/252530b9-e462-46c8-9362-2c7b584836c4"
+					(reference "R42")
 					(unit 1)
 				)
@@
 		(dnp no)
 		(fields_autoplaced yes)
-		(property "Reference" "R16"
+		(property "Reference" "R30"
 			(at 83.82 102.8699 0)
 			(show_name no)
@@
 		(instances
 			(project "MMS3_ESP32-C6"
-				(path "/712cea22-140d-4c92-923f-f4998caf3ecd/c085740e-6122-4df8-b6d1-901cece69bb5"
-					(reference "R16")
+				(path "/712cea22-140d-4c92-923f-f4998caf3ecd/252530b9-e462-46c8-9362-2c7b584836c4"
+					(reference "R30")
 					(unit 1)
 				)
@@
 		(instances
 			(project "MMS3_ESP32-C6"
-				(path "/712cea22-140d-4c92-923f-f4998caf3ecd/c085740e-6122-4df8-b6d1-901cece69bb5"
+				(path "/712cea22-140d-4c92-923f-f4998caf3ecd/252530b9-e462-46c8-9362-2c7b584836c4"
 					(reference "#PWR039")
 					(unit 1)
@@
 		(dnp yes)
 		(fields_autoplaced yes)
-		(property "Reference" "R22"
+		(property "Reference" "R32"
 			(at 167.64 105.4099 0)
 			(show_name no)
@@
 		(instances
 			(project "MMS3_ESP32-C6"
-				(path "/712cea22-140d-4c92-923f-f4998caf3ecd/c085740e-6122-4df8-b6d1-901cece69bb5"
-					(reference "R22")
+				(path "/712cea22-140d-4c92-923f-f4998caf3ecd/252530b9-e462-46c8-9362-2c7b584836c4"
+					(reference "R32")
 					(unit 1)
 				)
@@
 		(in_pos_files yes)
 		(dnp no)
-		(property "Reference" "U6"
+		(property "Reference" "U10"
 			(at 142.24 109.22 0)
 			(show_name no)
@@
 		(instances
 			(project "MMS3_ESP32-C6"
-				(path "/712cea22-140d-4c92-923f-f4998caf3ecd/c085740e-6122-4df8-b6d1-901cece69bb5"
-					(reference "U6")
+				(path "/712cea22-140d-4c92-923f-f4998caf3ecd/252530b9-e462-46c8-9362-2c7b584836c4"
+					(reference "U10")
 					(unit 1)
 				)
@@
 		(instances
 			(project "MMS3_ESP32-C6"
-				(path "/712cea22-140d-4c92-923f-f4998caf3ecd/c085740e-6122-4df8-b6d1-901cece69bb5"
+				(path "/712cea22-140d-4c92-923f-f4998caf3ecd/252530b9-e462-46c8-9362-2c7b584836c4"
 					(reference "#PWR043")
 					(unit 1)
@@
 		(instances
 			(project "MMS3_ESP32-C6"
-				(path "/712cea22-140d-4c92-923f-f4998caf3ecd/c085740e-6122-4df8-b6d1-901cece69bb5"
+				(path "/712cea22-140d-4c92-923f-f4998caf3ecd/252530b9-e462-46c8-9362-2c7b584836c4"
 					(reference "#PWR038")
 					(unit 1)

Commit message: backup commit
Parts:
- removed C16: 100nF, PCM_JLCPCB:C_0603, symbol PCM_JLCPCB-Capacitors:0603,100nF
- removed R30, R31, R32, R35, R40, R41, R42: 10kΩ, PCM_JLCPCB:R_0603, symbol PCM_JLCPCB-Resistors:0603,10kΩ
- added C51: 100nF, PCM_JLCPCB:C_0402, symbol PCM_JLCPCB-Capacitors:0402,100nF
- added R62, R63, R64, R65, R66, R67, R68: 10kΩ, PCM_JLCPCB:R_0402, symbol PCM_JLCPCB-Resistors:0402,10kΩ
Connections:
- net +3V3: now also C51.1, R66.1, R67.1, R68.1
- net A1: now also R64.1, R67.2
- net A2: now also R63.1, R66.2
- net GND: now also C51.2, R62.2, R63.2, R64.2, R65.2
- net I2C_Memory_addr: now also R65.1, R68.2
- net at U10.7 (WP): now also R62.1
