File: MMS3/IO.kicad_sch (KiCad schematic)
At the start: 5 parts, among them SW2 TC-6615Z-12.5-260

Commit message: backup commit
Parts:
- removed R24: 10kΩ, PCM_JLCPCB:R_0603, symbol PCM_JLCPCB-Resistors:0603,10kΩ
- removed R25, R26: 1kΩ, PCM_JLCPCB:R_0603, symbol PCM_JLCPCB-Resistors:0603,1kΩ
- removed SW2: TC-6615Z-12.5-260, Tact-sw:SW-TH_4P-L7.3-TC-6615Z-12.5-260, symbol Tact-sw:TC-6615Z-12.5-260
- added KEY1: TL2243, 2_tact_switch:KEY-TH_TL2243, symbol 2_tact_switch:TL2243
- added LED2: FixLed307, FixLed307:FixLed307, symbol FixLed307:FixLed307
- added R30, R31, R32, R35: 1kΩ, PCM_JLCPCB:R_0402, symbol PCM_JLCPCB-Resistors:0402,1kΩ
- added R40, R41: 10kΩ, PCM_JLCPCB:R_0402, symbol PCM_JLCPCB-Resistors:0402,10kΩ
Connections:
- net +3V3: now also KEY1.3, KEY1.4
- net GND: now also KEY1.0, LED2.2, LED2.4, R40.2, R41.2
- net GPIO4: now also KEY1.1, R41.1
- net GPIO5: now also R30.1
- net GPIO6: now also R31.1
- net GPIO7: now also R32.1
- net GPIO8: now also R35.1
- net GPIO9: now also KEY1.2, R40.1
- net at LED1.1: now also R31.2
- net at LED1.3: now also R30.2
- new net: LED2.1, R35.2
- new net: LED2.3, R32.2
Other:
- note removed: "External LED's"

Commit message: initial routing done
Connections:
- net GPIO4 is gone; now on net GPIO9: KEY1.1, R41.1
- net GPIO5 is gone; now on net GPIO8: R30.1
- net GPIO6 is gone; now on net GPIO7: R31.1
- net GPIO7: no longer R32.1
- net GPIO8: no longer R35.1
- net GPIO9: no longer KEY1.2, R40.1
- new net GPIO0: R32.1
- new net GPIO1: R35.1
- new net GPIO10: KEY1.2, R40.1
- no-connect marks 0 -> 2
Other:
- moved on the sheet: LED2A, LED2B, R32, R35

Commit message: eem, done?
Parts:
- LED1, LED2: now not fitted; now left out of the parts list
Connections:
- net +3V3: now also R31.1
- net GPIO7: no longer R31.1
