File: MMS3/MMS3_ESP32-C6.kicad_pcb (KiCad board)
At the start: 4 copper layers, 100 x 50 mm, 129 parts, among them J1 86093488324755V1LF, J2 AMASS XT60, J3 Program, J4 USB_C_Receptacle_USB2.0_16P, J5 Conn_Coaxial, J6 Conn_Coaxial, J7 AMASS XT60, J8 RJ45_LED_Shielded, J9 RJ45_LED_Shielded, SW1 SK12D07VG5, SW2 TC-6615Z-12.5-260, SW3 TC-6615Z-12.5-260, U1 TJA1044GTK_3Z, U10 AT24C256C, U11 ESP32-C6-WROOM-1-N4, U15 AMS1117-3.3, U2 TPS54560BDDA, U3 FSUSB42UMX, U4 TPD2EUSB30DRTR-TP, U5 TPD2EUSB30DRTR-TP, U6 TJA1044GTK_3Z, U7 FSUSB42UMX, U8 CH32V003FxPx, U9 TPD2EUSB30DRTR-TP, X1 X322525MOB4SI

Commit message: backup commit
Parts:
- removed C11, C16: 100nF, PCM_JLCPCB:C_0603
- removed C17: 10uF, PCM_JLCPCB:C_0603
- removed C18: 1uF, PCM_JLCPCB:C_0603
- removed J3: Program, Connector_PinHeader_2.54mm:PinHeader_1x03_P2.54mm_Vertical
- removed J6: Conn_Coaxial, Connector_Coaxial:SMA_Amphenol_901-143_Horizontal
- removed R42: 10kΩ, PCM_JLCPCB:R_0603
- removed S2: Tactile Button, 160gf, PCM_JLCPCB:SW_TS-1088-AR02016
- removed SW2: TC-6615Z-12.5-260, Tact-sw:SW-TH_4P-L7.3-TC-6615Z-12.5-260
- removed U8: CH32V003FxPx, PCM_JLCPCB:TSSOP-20_4.4x6.5mm_P0.65mm
- removed X1: X322525MOB4SI, PCM_JLCPCB:OSC-SMD_4P-L3.2-W2.5-BL
- added C1: 10nF, PCM_JLCPCB:C_0402, F.Cu at (157.6, 126.0)
- added C2: 10nF, PCM_JLCPCB:C_0402, F.Cu at (157.6, 121.4)
- added C22: 1.5pF, PCM_JLCPCB:C_0402, F.Cu at (186.0, 95.0)
- added C23: 100nF, PCM_JLCPCB:C_0402, F.Cu at (215.3, 100.0)
- added C25: 100nF, PCM_JLCPCB:C_0402, F.Cu at (237.6, 48.2)
- added C26: 10nF, PCM_JLCPCB:C_0402, F.Cu at (235.2, 44.0)
- added C27: 1uF, PCM_JLCPCB:C_0402, F.Cu at (233.4, 44.0)
- added C28: 100nF, PCM_JLCPCB:C_0402, F.Cu at (231.8, 48.2)
- added C29: 1uF, PCM_JLCPCB:C_0402, F.Cu at (230.8, 48.2)
- added C36: 10uF, PCM_JLCPCB:C_0402, F.Cu at (238.7, 48.2)
- added C37: 100nF, PCM_JLCPCB:C_0402, F.Cu at (154.0, 108.6)
- added C51: 100nF, PCM_JLCPCB:C_0402, F.Cu at (135.8, 106.7)
- added C52: 100nF, PCM_JLCPCB:C_0402, F.Cu at (236.0, 52.4)
- added C53: 100nF, PCM_JLCPCB:C_0402, F.Cu at (152.2, 98.2)
- added C54: 100nF, PCM_JLCPCB:C_0402, F.Cu at (224.1, 96.8)
- added C55: 100nF, PCM_JLCPCB:C_0402, F.Cu at (186.7, 107.8)
- added C57: 30pF, PCM_JLCPCB:C_0402, F.Cu at (160.0, 105.2)
- added C58: 30pF, PCM_JLCPCB:C_0402, F.Cu at (160.1, 101.0)
- added C59: 10uF, PCM_JLCPCB:C_0402, F.Cu at (232.8, 48.2)
- added C900: 100nF, PCM_JLCPCB:C_0402, F.Cu at (177.2, 113.0)
- added C902: 10uF, PCM_JLCPCB:C_0402, F.Cu at (177.2, 113.8)
- added C904: 1uF, PCM_JLCPCB:C_0402, F.Cu at (175.9, 113.5)
- added D301: Red, PCM_JLCPCB:D_0603, F.Cu at (173.0, 113.7)
- added FB1: ~, PCM_JLCPCB:FB_0805, F.Cu at (235.1, 47.7)
- added KEY1: TL2243, 2_tact_switch:KEY-TH_TL2243, F.Cu at (196.3, 108.7)
- added L5: 3.9nH,300mA, PCM_JLCPCB:L_0402, F.Cu at (187.9, 95.0)
- added LED2: FixLed307, FixLed307:FixLed307, F.Cu at (195.8, 101.6)
- added Q1: MMBT3904 100-300, PCM_JLCPCB:Q_SOT-23, F.Cu at (169.8, 101.5)
- added Q2: MMBT3904 100-300, PCM_JLCPCB:Q_SOT-23, F.Cu at (169.8, 104.9)
- added R2: 220Ω, PCM_JLCPCB:R_0402, F.Cu at (241.2, 111.6)
- added R308: 1kΩ, PCM_JLCPCB:R_0402, F.Cu at (175.1, 113.5)
- added R48: 0Ω, PCM_JLCPCB:R_0402, F.Cu at (152.5, 106.5)
- added R49: 510Ω, PCM_JLCPCB:R_0402, F.Cu at (154.2, 106.5)
- added R5: 33kΩ, PCM_JLCPCB:R_0402, F.Cu at (157.6, 128.2)
- added R50: 22Ω, PCM_JLCPCB:R_0402, F.Cu at (147.7, 103.3)
- added R51: 22Ω, PCM_JLCPCB:R_0402, F.Cu at (147.7, 104.1)
- added R52: 10kΩ, PCM_JLCPCB:R_0402, F.Cu at (147.7, 102.2)
- added R53: 10kΩ, PCM_JLCPCB:R_0402, F.Cu at (153.5, 98.0)
- added R54: 10kΩ, PCM_JLCPCB:R_0402, F.Cu at (147.7, 101.4)
- added R55: 10kΩ, PCM_JLCPCB:R_0402, F.Cu at (149.4, 98.6)
- added R56: 10kΩ, PCM_JLCPCB:R_0402, F.Cu at (148.6, 98.6)
- added R6: 33kΩ, PCM_JLCPCB:R_0402, F.Cu at (157.6, 119.4)
- added R62: 10kΩ, PCM_JLCPCB:R_0402, F.Cu at (138.6, 104.0)
- added R63: 10kΩ, PCM_JLCPCB:R_0402, F.Cu at (140.3, 108.5)
- added R64: 10kΩ, PCM_JLCPCB:R_0402, F.Cu at (141.2, 108.5)
- added R65: 10kΩ, PCM_JLCPCB:R_0402, F.Cu at (139.4, 108.5)
- added R66: 10kΩ, PCM_JLCPCB:R_0402, F.Cu at (140.3, 110.5)
- added R67: 10kΩ, PCM_JLCPCB:R_0402, F.Cu at (141.2, 110.5)
- added R68: 10kΩ, PCM_JLCPCB:R_0402, F.Cu at (139.4, 110.5)
- added R902: 22Ω, PCM_JLCPCB:R_0402, F.Cu at (178.4, 108.5)
- added R903: 22Ω, PCM_JLCPCB:R_0402, F.Cu at (178.4, 107.7)
- added R906: 22Ω, PCM_JLCPCB:R_0402, F.Cu at (172.7, 108.0)
- added R907: 22Ω, PCM_JLCPCB:R_0402, F.Cu at (172.7, 108.8)
- added SW4: TC-6615Z-12.5-260, Tact-sw:SW-TH_4P-L7.3-TC-6615Z-12.5-260, F.Cu at (242.9, 81.6)
- added U12: TCA9555RTWR, I2C_GPIO:HVQFN-24_L4.0-W4.0-P0.50-BL-EP2.6, F.Cu at (186.7, 111.4)
- added U13: CH340G, PCM_JLCPCB:SOIC-16_3.9x9.9mm_P1.27mm, F.Cu at (177.7, 103.4)
- added U14: XT25F128FWOIGT-W, SPI_flash:WSON-8_L6.0-W5.0-P1.27-BL-EP, F.Cu at (151.6, 111.6)
- added U302: CH334P, Package_DFN_QFN:QFN-16-1EP_3x3mm_P0.5mm_EP1.7x1.7mm, F.Cu at (175.8, 110.3)
- added X2: 40MHz, 15pF, PCM_JLCPCB:OSC-SMD_4P-L3.2-W2.5-BL_SIT8008BI, F.Cu at (160.1, 103.1)
- added X3: X322512MSB4SI, PCM_JLCPCB:CRYSTAL-SMD_4P-L3.2-W2.5-BL, F.Cu at (184.7, 103.8)
- added Y900: Crystal_GND24, Crystal:Crystal_SMD_3225-4Pin_3.2x2.5mm, F.Cu at (180.5, 111.1)
- C12: value 12pF -> 100nF; footprint PCM_JLCPCB:C_0603 -> PCM_JLCPCB:C_0402
- C13: value 12pF -> 10nF; footprint PCM_JLCPCB:C_0603 -> PCM_JLCPCB:C_0402
- C14: value 10nF -> 20pF; footprint PCM_JLCPCB:C_0603 -> PCM_JLCPCB:C_0402
- C15: value 100nF -> 20pF; footprint PCM_JLCPCB:C_0603 -> PCM_JLCPCB:C_0402
- C19: value 100nF -> 1uF; footprint PCM_JLCPCB:C_0603 -> PCM_JLCPCB:C_0402
- J5: footprint Connector_Coaxial:U.FL_Molex_MCRF_73412-0110_Vertical -> Connector_Coaxial:SMA_Amphenol_901-143_Horizontal
- R16, R17, R23, R24, R27, R40, R41: footprint PCM_JLCPCB:R_0603 -> PCM_JLCPCB:R_0402
- R18, R19, R20, R21: value 0Ω -> 22Ω; footprint PCM_JLCPCB:R_0603 -> PCM_JLCPCB:R_0402
- R22, R43, R44, R45, R46, R47: value 10kΩ -> 0Ω; footprint PCM_JLCPCB:R_0603 -> PCM_JLCPCB:R_0402
- R25, R26: value 1kΩ -> 5.1kΩ; footprint PCM_JLCPCB:R_0603 -> PCM_JLCPCB:R_0402
- R28, R29: value 5.1kΩ -> 10kΩ; footprint PCM_JLCPCB:R_0603 -> PCM_JLCPCB:R_0402
- R30, R31, R32, R35: value 10kΩ -> 1kΩ; footprint PCM_JLCPCB:R_0603 -> PCM_JLCPCB:R_0402
- TP1, TP2, TP3, TP4: moved to B.Cu
- U11: value ESP32-C6-WROOM-1-N4 -> ESP32-C6_C5364646; footprint ESPRESSIF_ESP32-C6-WROOM-1-N4:WIRELM-SMD_ESP32-C6-WROOM-1 -> ESP32-C6-QFN40:QFN-40_L5.0-W5.0-P0.40-TL-EP3.3
- moved U10 114.6 mm to (139.3, 109.8), turned to 90 degrees
- moved R4 100.1 mm to (248.8, 62.6)
- moved R28 91.8 mm to (166.4, 102.5)
- moved R29 91.8 mm to (166.4, 104.8)
- moved R47 91.4 mm to (149.0, 106.5), turned to -90 degrees
- moved R3 88.6 mm to (241.2, 107.7)
- moved R46 87.3 mm to (153.3, 106.5), turned to -90 degrees
- moved C19 86.8 mm to (153.5, 97.2)
- moved R27 80.4 mm to (184.3, 123.1), turned to 180 degrees
- moved R44 79.0 mm to (150.1, 106.5), turned to -90 degrees
- moved R45 78.8 mm to (151.7, 106.5), turned to -90 degrees
- moved U3 78.5 mm to (158.0, 114.6)
- moved R43 77.2 mm to (150.9, 106.5), turned to -90 degrees
- moved R16 72.5 mm to (172.4, 111.0), turned to 180 degrees
- moved U9 71.8 mm to (181.5, 122.6), turned to 90 degrees
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Connections:
- C12 pad 1: /GPIO_Expander/OSCI -> /USBC_CONN/VBUS
- C13 pad 1: /GPIO_Expander/OSCO -> Net-(J4-SHIELD)
- C14 pad 1: Net-(J4-SHIELD) -> /UART_Programmer/XI
- C15 pad 1: /USBC_CONN/VBUS -> /UART_Programmer/XO
- C19 pad 1: +3V3 -> /ESP32-C6/EN
- J4 pad A6: /Bypass_jumper/USB2.D+ -> /USB switch1/USB_OUT2.D+
- J4 pad A7: /Bypass_jumper/USB2.D- -> /USB switch1/USB_OUT2.D-
- J4 pad B6: /Bypass_jumper/USB2.D+ -> /USB switch1/USB_OUT2.D+
- J4 pad B7: /Bypass_jumper/USB2.D- -> /USB switch1/USB_OUT2.D-
- R16 pad 1: /Bypass_jumper/USB1.D- -> /USB HUB/USBIN1_R.D+
- R16 pad 2: /ESP32-C6 Wrapper/ESP D- -> /USB HUB/USBIN1.D+
- R17 pad 1: /Bypass_jumper/USB1.D+ -> /USB HUB/USBIN1_R.D-
- R17 pad 2: /ESP32-C6 Wrapper/ESP D+ -> /USB HUB/USBIN1.D-
- R18 pad 1: /Bypass_jumper/USB1.D+ -> /USB HUB/USBBYP.D+
- R18 pad 2: /Bypass_jumper/bypass_D+ -> /USB HUB/USBIN1.D+
- R19 pad 1: /Bypass_jumper/USB1.D- -> /USB HUB/USBBYP.D-
- R19 pad 2: /Bypass_jumper/bypass_D- -> /USB HUB/USBIN1.D-
- R20 pad 1: /Bypass_jumper/bypass_D+ -> /USB HUB/USBBYP.D-
- R20 pad 2: /Bypass_jumper/USB2.D+ -> /ESP32-C6/USB.D-
- R21 pad 1: /Bypass_jumper/bypass_D- -> /USB HUB/USBBYP.D+
- R21 pad 2: /Bypass_jumper/USB2.D- -> /ESP32-C6/USB.D+
- R22 pad 1: +3V3 -> /ESP32-C6/XTAL_P.
- R22 pad 2: /ChainBus + ALtmode/Altmode1 -> /ESP32-C6/XTAL_P
- R23 pad 2: /GPIO_Expander/PD7 -> /GPIO_Expander/A0
- R24 pad 1: /GPIO_Expander/GPIO6 -> +3V3
- R24 pad 2: GND -> /GPIO_Expander/A2
- R25 pad 1: /GPIO_Expander/GPIO4 -> /USBC_CONN/CC1
- R25 pad 2: Net-(LED1-Pad3) -> GND
- R26 pad 1: /GPIO_Expander/GPIO5 -> /USBC_CONN/CC2
- R26 pad 2: Net-(LED1-Pad1) -> GND
- R28 pad 1: /USBC_CONN/CC2 -> /UART_Programmer/~{DTR}
- R28 pad 2: GND -> Net-(Q1-B)
- R29 pad 1: /USBC_CONN/CC1 -> /UART_Programmer/~{RTS}
- R29 pad 2: GND -> Net-(Q2-B)
- R30 pad 1: Net-(U10-WP) -> /User IO/GPIO5
- R30 pad 2: GND -> Net-(LED1-Pad3)
- R31 pad 1: +3V3 -> /User IO/GPIO6
- R31 pad 2: /I2C_Flash/A2 -> Net-(LED1-Pad1)
- R32 pad 1: /I2C_Flash/A2 -> /User IO/GPIO7
- R32 pad 2: GND -> Net-(LED2-Pad3)
- R35 pad 1: +3V3 -> /User IO/GPIO8
- R35 pad 2: /I2C_Flash/A1 -> Net-(LED2-Pad1)
- R40 pad 1: /I2C_Flash/A1 -> /User IO/GPIO9
- R41 pad 1: +3V3 -> /User IO/GPIO4
- R41 pad 2: /I2C_Flash/A0 -> GND
- R43 pad 1: /ESP32-C6 Wrapper/ESP32-C6/EN -> /ESP32-C6/ESP_SPIWP
- R43 pad 2: +3V3 -> /ESP32-C6/SPIWP
- R44 pad 1: /ChainBus + ALtmode/Chainbus_addr5 -> /ESP32-C6/ESP_SPIQ
- R44 pad 2: +3V3 -> /ESP32-C6/SPIQ
- R45 pad 1: /ChainBus + ALtmode/Chainbus_addr8 -> /ESP32-C6/ESP_SPIHD
- R45 pad 2: +3V3 -> /ESP32-C6/SPIHD
- R46 pad 1: /ChainBus + ALtmode/Chainbus.RX -> /ESP32-C6/ESP_SPID
- R46 pad 2: +3V3 -> /ESP32-C6/SPID
- R47 pad 1: /ChainBus + ALtmode/Chainbus.TX -> /ESP32-C6/ESP_SPICS0
- R47 pad 2: GND -> /ESP32-C6/SPICS0
- R8 pad 1: /Slide-SW/SEL -> /USB switch/SEL
- SW3 pad 1: /ESP32-C6 Wrapper/ESP32-C6/EN -> /ESP32-C6/EN
- TP1 pad 1: /ChainBus + ALtmode/Altmode2 -> /CAN2.TX
- TP2 pad 1: /ChainBus + ALtmode/Altmode3 -> /CAN2.RX
- TP3 pad 1: /ChainBus + ALtmode/Altmode5 -> /CAN1.TX
- TP4 pad 1: /ChainBus + ALtmode/Altmode4 -> /CAN1.RX
- U1 pad 1: /ChainBus + ALtmode/Altmode2 -> /CAN2.TX
- U1 pad 4: /ChainBus + ALtmode/Altmode3 -> /CAN2.RX
- U11 pad 1: +3V3 -> /ESP32-C6/ANT
- U11 pad 10: /ChainBus + ALtmode/Chainbus_addr8 -> /ChainBus + ALtmode/Chainbus.RX
- U11 pad 11: /ChainBus + ALtmode/Chainbus_addr7 -> /ChainBus + ALtmode/Chainbus.TX
- U11 pad 12: /ChainBus + ALtmode/Chainbus_addr6 -> /ChainBus + ALtmode/Chainbus.SDA
- U11 pad 13: /ESP32-C6 Wrapper/ESP D- -> /ChainBus + ALtmode/Chainbus.SCL
- U11 pad 14: /ESP32-C6 Wrapper/ESP D+ -> /ChainBus + ALtmode/Chainbus_addr5
- U11 pad 15: /ChainBus + ALtmode/Chainbus_addr5 -> /ChainBus + ALtmode/Chainbus_addr8
- U11 pad 16: /ChainBus + ALtmode/Chainbus.SCK -> /ChainBus + ALtmode/Chainbus_addr7
- U11 pad 17: /ChainBus + ALtmode/Chainbus.MOSI -> /ChainBus + ALtmode/Chainbus_addr6
- U11 pad 18: /ChainBus + ALtmode/Chainbus.MISO -> /ESP32-C6/GPIO12
- U11 pad 19: /ChainBus + ALtmode/Altmode5 -> /ESP32-C6/GPIO13
- U11 pad 2: GND -> /ESP32-C6/VCC_RF
- U11 pad 20: /ChainBus + ALtmode/Altmode4 -> /ESP32-C6/ESP_SPICS0
- U11 pad 21: /ChainBus + ALtmode/Chainbus.CS -> /ESP32-C6/ESP_SPIQ
- U11 pad 22: unconnected-(U11-NC-Pad22) -> /ESP32-C6/ESP_SPIWP
- U11 pad 23: /ChainBus + ALtmode/Altmode3 -> /ChainBus + ALtmode/Altmode4
- U11 pad 24: /ChainBus + ALtmode/Altmode2 -> /ESP32-C6/ESP_SPIHD
- U11 pad 25: /ChainBus + ALtmode/Altmode1 -> /ESP32-C6/ESP_CSPICLK
- U11 pad 26: /ChainBus + ALtmode/Chainbus_addr4 -> /ESP32-C6/ESP_SPID
- U11 pad 27: /ChainBus + ALtmode/Chainbus_addr3 -> /ChainBus + ALtmode/Altmode3
- U11 pad 28: GND -> +3V3
- U11 pad 29: GND -> /ESP32-C6/ESP_TX
- U11 pad 3: /ESP32-C6 Wrapper/ESP32-C6/EN -> /ESP32-C6/VCC_RF
- U11 pad 30: GND -> /ESP32-C6/UART0.RX
- U11 pad 31: GND -> /ChainBus + ALtmode/Chainbus.SCK
- U11 pad 32: GND -> /ChainBus + ALtmode/Chainbus.MOSI
- U11 pad 33: GND -> /ChainBus + ALtmode/Chainbus.MISO
- U11 pad 34: GND -> /ChainBus + ALtmode/Altmode1
- U11 pad 35: GND -> /ChainBus + ALtmode/Altmode2
- U11 pad 36: GND -> /ChainBus + ALtmode/Chainbus.CS
- U11 pad 37: GND -> +3V3
- U11 pad 4: /ChainBus + ALtmode/Chainbus.RX -> /ESP32-C6/EN
- U11 pad 5: /ChainBus + ALtmode/Chainbus.TX -> +3V3
- U11 pad 6: /ChainBus + ALtmode/Chainbus.SDA -> /ChainBus + ALtmode/Chainbus_addr2
- U11 pad 7: /ChainBus + ALtmode/Chainbus.SCL -> /ChainBus + ALtmode/Chainbus_addr1
- U11 pad 8: /ChainBus + ALtmode/Chainbus_addr1 -> /ChainBus + ALtmode/Chainbus_addr3
- U11 pad 9: /ChainBus + ALtmode/Chainbus_addr2 -> /ChainBus + ALtmode/Chainbus_addr4
- U6 pad 1: /ChainBus + ALtmode/Altmode5 -> /CAN1.TX
- U6 pad 4: /ChainBus + ALtmode/Altmode4 -> /CAN1.RX
- U7 pad 1: /Bypass_jumper/USB1.D+ -> /USB HUB/USBIN1.D+
- U7 pad 2: /Bypass_jumper/USB1.D- -> /USB HUB/USBIN1.D-
- U7 pad 6: /Bypass_jumper/USB2.D- -> /USB switch1/USB_OUT2.D-
- U7 pad 7: /Bypass_jumper/USB2.D+ -> /USB switch1/USB_OUT2.D+
- U9 pad 1: /Bypass_jumper/USB2.D- -> /USB switch1/USB_OUT2.D-
- U9 pad 2: /Bypass_jumper/USB2.D+ -> /USB switch1/USB_OUT2.D+
Routing:
- net /ESP32-C6/USB.D+: track 0.00 -> 41.3 mm, vias 0 -> 2
- net /ESP32-C6/USB.D-: track 0.00 -> 40.2 mm, vias 0 -> 2
- net /ESP32-C6/ANT: track 0.00 -> 32.3 mm
- net /USB switch1/USB_OUT2.D-: track 0.00 -> 28.6 mm
- net /USB switch1/USB_OUT2.D+: track 0.00 -> 27.4 mm
- net /CAN_TR.kicad_sch/CAN.-: track 0.00 -> 25.5 mm
- net /CAN_TR.kicad_sch/CAN.+: track 0.00 -> 25.4 mm
- net /CAN_TR.kicad_sch1/CAN.-: track 0.00 -> 24.9 mm
- net /MMS_CONNECTOR_UPSTREAM/USB_MMS_CONN.D-: track 0.00 -> 22.8 mm
- net /CAN_TR.kicad_sch1/CAN.+: track 0.00 -> 22.1 mm
- net /MMS_CONNECTOR_DOWNSTREAM/USB_MMS_CONN.D-: track 0.00 -> 21.2 mm, vias 0 -> 2
- net /MMS_CONNECTOR_UPSTREAM/USB_MMS_CONN.D+: track 0.00 -> 20.1 mm
- net /MMS_CONNECTOR_DOWNSTREAM/USB_MMS_CONN.D+: track 0.00 -> 16.5 mm, vias 0 -> 2
- net /ESP32-C6/SPID: track 0.00 -> 8.61 mm
- net /USB switch/USB_OUT2.D-: track 0.00 -> 7.73 mm, vias 0 -> 2
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Other:
- board text added: "5w keept"
- board text added: "RF line"

Commit message: working commit
Parts:
- removed C36: 10uF, PCM_JLCPCB:C_0402
- removed R22: 0Ω, PCM_JLCPCB:R_0402
- removed U14: XT25F128FWOIGT-W, SPI_flash:WSON-8_L6.0-W5.0-P1.27-BL-EP
- added C17: 2.2pF, PCM_JLCPCB:C_0402, F.Cu at (162.0, 107.9)
- added C18: 3.3pF, PCM_JLCPCB:C_0402, F.Cu at (159.4, 107.9)
- added L2: 15nH,300mA, PCM_JLCPCB:L_0402, F.Cu at (156.6, 111.1)
- added L3: 2n, PCM_JLCPCB:C_0402, F.Cu at (160.7, 107.4)
- added R42: 0Ω, PCM_JLCPCB:R_0402, F.Cu at (186.7, 94.6)
- added R57: 0Ω, PCM_JLCPCB:R_0402, F.Cu at (185.0, 95.1)
- added R58: 0Ω, PCM_JLCPCB:R_0402, F.Cu at (188.5, 95.1)
- added U8: ZD25Q128CSIGT, spi_flash:SOP-8_L5.3-W5.3-P1.27-LS7.9-BL, F.Cu at (145.2, 103.0)
- moved C26 101.4 mm to (157.2, 108.8)
- moved C27 101.3 mm to (155.5, 108.8)
- moved C52 101.0 mm to (150.2, 105.7), turned to 180 degrees
- moved C25 96.9 mm to (159.9, 106.0), turned to -20 degrees
- moved FB1 92.3 mm to (161.6, 103.5), turned to 90 degrees
- moved C59 90.4 mm to (159.5, 101.1), turned to 90 degrees
- moved C28 90.1 mm to (160.3, 102.9)
- moved C29 88.2 mm to (160.3, 101.1), turned to 90 degrees
- moved R19 52.6 mm to (249.1, 100.7)
- moved R20 52.6 mm to (249.1, 98.1)
- moved R18 52.6 mm to (247.9, 100.7)
- moved R21 52.6 mm to (247.9, 98.1)
- moved R68 50.6 mm to (184.9, 88.3), turned to 180 degrees
- moved R66 50.2 mm to (184.9, 87.4), turned to 180 degrees
- moved R67 49.8 mm to (184.9, 86.5), turned to 180 degrees
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Connections:
- net Net-(C20-Pad1) renamed /ESP32-C6/More_RF
- C22 pad 1: Net-(C18-Pad1) -> /ESP32-C6/RF
- J5 pad 1: Net-(J5-In) -> /ESP32-C6/ANT_CN
- TP1 pad 1: /CAN2.TX -> /ChainBus + ALtmode/Altmode1
- TP2 pad 1: /CAN2.RX -> /ChainBus + ALtmode/Altmode2
- TP3 pad 1: /CAN1.TX -> /ChainBus + ALtmode/Altmode3
- TP4 pad 1: /CAN1.RX -> /ChainBus + ALtmode/Altmode4
- U1 pad 1: /CAN2.TX -> /ChainBus + ALtmode/Altmode1
- U1 pad 4: /CAN2.RX -> /ChainBus + ALtmode/Altmode2
- U11 pad 34: /ChainBus + ALtmode/Altmode1 -> /ChainBus + ALtmode/Altmode2
- U11 pad 35: /ChainBus + ALtmode/Altmode2 -> /ChainBus + ALtmode/Altmode1
- U6 pad 1: /CAN1.TX -> /ChainBus + ALtmode/Altmode3
- U6 pad 4: /CAN1.RX -> /ChainBus + ALtmode/Altmode4
Routing:
- net +12V stby: track 154.5 -> 45.7 mm
- net +5V: track 98.8 -> 0.00 mm, vias 4 -> 0
- net GND: track 108.1 -> 24.2 mm, vias 142 -> 158
- net /ESP32-C6/ANT: track 32.3 -> 3.51 mm
- net /ESP32-C6/More_RF: track 0.00 -> 28.7 mm
- net /ESP32-C6/USB.D+: track 41.3 -> 19.1 mm, vias 2 -> 1
- net /ESP32-C6/USB.D-: track 40.2 -> 19.6 mm, vias 2 -> 1
- net /ChainBus + ALtmode/Chainbus.TX: track 0.00 -> 17.7 mm
- net /ChainBus + ALtmode/Chainbus.SDA: track 0.00 -> 17.4 mm
- net /ChainBus + ALtmode/Chainbus.RX: track 0.00 -> 16.7 mm, vias 0 -> 2
- net /ChainBus + ALtmode/Chainbus.SCL: track 0.00 -> 13.5 mm
- net +3V3: track 1.22 -> 13.7 mm, vias 0 -> 6
- net /ESP32-C6/ANT_CN: track 0.00 -> 7.05 mm
- net /ESP32-C6/VCC_RF: track 0.00 -> 6.48 mm
- net /ESP32-C6/XTAL_N: track 0.00 -> 6.38 mm
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- added copper zone on F.Cu, net +3V3

Commit message: initial routing done
Parts:
- removed R21: 22Ω, PCM_JLCPCB:R_0402
- removed SW4: TC-6615Z-12.5-260, Tact-sw:SW-TH_4P-L7.3-TC-6615Z-12.5-260
- added D6: 1N5819WS, PCM_JLCPCB:D_SOD-323, F.Cu at (190.4, 115.8)
- added D7: 1N5819WS, PCM_JLCPCB:D_SOD-323, F.Cu at (188.5, 115.8)
- added G***: LOGO, LOGO, B.Cu at (176.6, 111.4)
- added R59: 10kΩ, PCM_JLCPCB:R_0402, F.Cu at (181.0, 85.8)
- added R60: 10kΩ, PCM_JLCPCB:R_0402, F.Cu at (181.0, 86.5)
- added R61: 10kΩ, PCM_JLCPCB:R_0402, F.Cu at (185.7, 108.4)
- added REF**: WEEE-Logo_4.2x6mm_SilkScreen, Symbol:WEEE-Logo_4.2x6mm_SilkScreen, B.Cu at (133.0, 100.3)
- moved R4 81.3 mm to (186.1, 114.4), turned to 90 degrees
- moved R20 77.7 mm to (171.8, 106.2)
- moved R19 77.6 mm to (171.9, 108.0), turned to -90 degrees
- moved R18 75.6 mm to (172.7, 108.0), turned to -90 degrees
- moved G*** 70.4 mm to (137.2, 98.7)
- moved G*** 63.1 mm to (145.0, 103.4)
- moved TP1 58.0 mm to (141.7, 97.4)
- moved R2 57.6 mm to (183.7, 114.4), turned to 90 degrees
- moved R3 57.1 mm to (184.5, 114.4), turned to 90 degrees
- moved R1 56.5 mm to (185.3, 114.4), turned to 90 degrees
- moved TP2 56.5 mm to (142.5, 100.7)
- moved TP4 54.9 mm to (138.9, 99.8)
- moved TP3 53.8 mm to (136.9, 100.5)
- moved C54 48.5 mm to (175.6, 98.2), turned to -90 degrees
- moved C23 35.6 mm to (180.0, 104.6), turned to 180 degrees
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Connections:
- KEY1 pad 1: /User IO/GPIO4 -> /GPIO_Expander/GPIO9
- KEY1 pad 2: /User IO/GPIO9 -> /GPIO_Expander/GPIO10
- Q2 pad 3: /ChainBus + ALtmode/Chainbus_addr8 -> /ChainBus + ALtmode/Chainbus_addr7
- R18 pad 1: /USB HUB/USBBYP.D+ -> /ESP32-C6/USB.D+
- R30 pad 1: /User IO/GPIO5 -> /GPIO_Expander/GPIO8
- R31 pad 1: /User IO/GPIO6 -> /GPIO_Expander/GPIO7
- R32 pad 1: /User IO/GPIO7 -> /GPIO_Expander/GPIO0
- R35 pad 1: /User IO/GPIO8 -> /GPIO_Expander/GPIO1
- R40 pad 1: /User IO/GPIO9 -> /GPIO_Expander/GPIO10
- R41 pad 1: /User IO/GPIO4 -> /GPIO_Expander/GPIO9
- R52 pad 1: /ChainBus + ALtmode/Chainbus_addr8 -> /ChainBus + ALtmode/Chainbus_addr7
- R54 pad 1: /ChainBus + ALtmode/Chainbus_addr5 -> /ChainBus + ALtmode/Chainbus_addr8
- TP1 pad 1: /ChainBus + ALtmode/Altmode1 -> /ChainBus + ALtmode/Altmode4
- TP2 pad 1: /ChainBus + ALtmode/Altmode2 -> /ChainBus + ALtmode/Altmode3
- TP3 pad 1: /ChainBus + ALtmode/Altmode3 -> /ChainBus + ALtmode/Altmode1
- TP4 pad 1: /ChainBus + ALtmode/Altmode4 -> /ChainBus + ALtmode/Altmode2
- U1 pad 1: /ChainBus + ALtmode/Altmode1 -> /ChainBus + ALtmode/Altmode4
- U1 pad 4: /ChainBus + ALtmode/Altmode2 -> /ChainBus + ALtmode/Altmode3
- U11 pad 14: /ChainBus + ALtmode/Chainbus_addr5 -> /ChainBus + ALtmode/Chainbus_addr8
- U11 pad 15: /ChainBus + ALtmode/Chainbus_addr8 -> /ChainBus + ALtmode/Chainbus_addr7
- U11 pad 16: /ChainBus + ALtmode/Chainbus_addr7 -> /ChainBus + ALtmode/Chainbus_addr6
- U11 pad 17: /ChainBus + ALtmode/Chainbus_addr6 -> /ChainBus + ALtmode/Chainbus_addr5
- U11 pad 6: /ChainBus + ALtmode/Chainbus_addr2 -> /ChainBus + ALtmode/Chainbus_addr1
- U11 pad 7: /ChainBus + ALtmode/Chainbus_addr1 -> /ChainBus + ALtmode/Chainbus_addr2
- U12 pad 1: /GPIO_Expander/GPIO0 -> /GPIO_Expander/A2
- U12 pad 10: /GPIO_Expander/GPIO8 -> /Select_GPIO
- U12 pad 11: /GPIO_Expander/GPIO9 -> /GPIO_Expander/GPIO7
- U12 pad 12: /GPIO_Expander/GPIO10 -> /GPIO_Expander/GPIO8
- U12 pad 13: /GPIO_Expander/GPIO11 -> /GPIO_Expander/GPIO9
- U12 pad 14: unconnected-(U12-P14-Pad14) -> /GPIO_Expander/GPIO10
- U12 pad 15: /GPIO_Expander/A0 -> /GPIO_Expander/GPIO11
- U12 pad 16: GND -> /GPIO_Expander/GPIO12
- U12 pad 17: /GPIO_Expander/A2 -> /GPIO_Expander/A0
- U12 pad 2: /GPIO_Expander/GPIO1 -> /GPIO_Expander/A1
- U12 pad 23: GND -> /GPIO_Expander/A1
- U12 pad 3: /GPIO_Expander/GPIO2 -> /GPIO_Expander/GPIO0
- U12 pad 4: /GPIO_Expander/GPIO3 -> /GPIO_Expander/GPIO1
- U12 pad 5: /GPIO_Expander/GPIO4 -> /RJ45_UP_TX1
- U12 pad 6: /GPIO_Expander/GPIO5 -> /RJ45_DWN_RX1
- U12 pad 7: /GPIO_Expander/GPIO6 -> /RJ45_DWN_TX1
- U12 pad 8: /GPIO_Expander/GPIO7 -> /RJ45_UP_RX1
- U6 pad 1: /ChainBus + ALtmode/Altmode3 -> /ChainBus + ALtmode/Altmode1
- U6 pad 4: /ChainBus + ALtmode/Altmode4 -> /ChainBus + ALtmode/Altmode2
Routing:
- net +3V3: track 13.7 -> 219.7 mm, vias 6 -> 24
- net +5V: track 0.00 -> 106.1 mm, vias 0 -> 20
- net +12V stby: track 45.7 -> 151.4 mm
- net GND: track 24.2 -> 102.9 mm, vias 158 -> 263
- net /ChainBus + ALtmode/Chainbus.SCL: track 13.5 -> 74.3 mm, vias 0 -> 4
- net /ChainBus + ALtmode/Chainbus.SDA: track 17.4 -> 78.1 mm, vias 0 -> 4
- net Net-(J9-~-Pad12): track 0.00 -> 51.9 mm, vias 0 -> 3
- net /ESP32-C6/EN: track 0.96 -> 51.0 mm, vias 1 -> 6
- net /ESP32-C6/UART0.TX: track 0.00 -> 44.6 mm, vias 0 -> 2
- net /ESP32-C6/UART0.RX: track 1.26 -> 44.2 mm, vias 0 -> 2
- net /USB switch/SEL: track 0.00 -> 41.3 mm, vias 0 -> 3
- net /ChainBus + ALtmode/Chainbus_addr7: track 0.00 -> 40.4 mm, vias 0 -> 4
- net /ChainBus + ALtmode/Chainbus_addr1: track 1.97 -> 41.1 mm, vias 1 -> 2
- net /ChainBus + ALtmode/Chainbus_addr2: track 1.85 -> 37.2 mm, vias 1 -> 2
- net /ChainBus + ALtmode/Altmode1: track 1.95 -> 36.8 mm, vias 1 -> 3
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- removed copper zone on F.Cu, net +3V3
Other:
- board text added: "LED -> USB ChainLink"
- board text removed: "Boot"
- board text removed: "LED high: USB from ChainLink"
- board text removed: "USB-SW"

Commit message: routing done
Parts:
- removed REF**: WEEE-Logo_4.2x6mm_SilkScreen, Symbol:WEEE-Logo_4.2x6mm_SilkScreen
- added D8: TPD1E0B04DPYR, RF_TVS:X1SON-2_L1.0-W0.6-P0.65-BI, F.Cu at (189.1, 95.1)
- moved U7 2.13 mm to (164.4, 111.6)
- moved C8 1.60 mm to (166.3, 111.1), turned to 90 degrees
- moved R42 1.28 mm to (185.4, 94.6)
- moved R57 1.28 mm to (183.7, 95.1)
- moved R58 1.28 mm to (187.2, 95.1)
- moved Y900 1.25 mm to (181.4, 110.6), turned to 0 degrees
- moved D5 0.07 mm to (168.9, 111.7)
- turned U4 to 180 degrees
Routing:
- net +3V3: track 219.7 -> 244.9 mm
- net /ESP32-C6/UART0.RX: track 44.2 -> 49.5 mm
- net /ESP32-C6/UART0.TX: track 44.6 -> 49.6 mm
- net /MMS_CONNECTOR_DOWNSTREAM/USB_MMS_CONN.D+: track 16.5 -> 20.6 mm, vias 2 -> 0
- net Net-(U302-XI): track 2.47 -> 6.21 mm
- net /MMS_CONNECTOR_UPSTREAM/USB_MMS_CONN.D-: track 22.8 -> 20.4 mm
- net /USB switch/USB_OUT2.D+: track 6.18 -> 8.42 mm
- net +12V stby: track 151.4 -> 153.3 mm
- net /USB switch/SEL: track 41.3 -> 43.1 mm
- net Net-(U7-~{OE}): track 5.77 -> 4.07 mm, vias 2 -> 0
- net GND: track 102.9 -> 101.3 mm, vias 263 -> 274
- net /USB switch1/USB_OUT2.D-: track 28.6 -> 27.0 mm
- net /ESP32-C6/ANT_CN: track 7.05 -> 8.33 mm
- net /USB switch1/USB_OUT2.D+: track 27.4 -> 26.4 mm
- net /USB HUB/USBIN1.D+: track 13.1 -> 12.3 mm
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Other:
- board text added: "LED -> USB from ChainLink"
- board text removed: "5w keept"
- board text removed: "LED -> USB ChainLink"
- board text removed: "RF line"

Commit message: eem, done?
Parts:
- R50, R51: value 22Ω -> 0Ω
- moved C54 13.8 mm to (189.3, 96.2), turned to 0 degrees
- moved C15 9.55 mm to (179.5, 108.0), turned to 180 degrees
- moved C14 9.16 mm to (179.9, 104.2)
- moved X3 9.16 mm to (179.9, 106.0)
- moved R28 7.78 mm to (168.1, 103.7)
- moved C23 5.09 mm to (181.9, 99.9), turned to 90 degrees
- moved U13 5.06 mm to (186.1, 101.8), turned to 0 degrees
- moved Q1 3.57 mm to (170.2, 102.5), turned to 90 degrees
- moved Q2 3.47 mm to (173.6, 102.5), turned to 90 degrees
- moved R903 2.40 mm to (176.0, 106.0), turned to -90 degrees
- moved R902 1.81 mm to (176.8, 106.0), turned to -90 degrees
- moved R29 1.01 mm to (175.8, 101.0)
- moved D8 1.01 mm to (189.1, 94.1), turned to -90 degrees
- moved C37 0.66 mm to (148.3, 106.0)
- moved R50 0.16 mm to (153.6, 100.2)
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Connections:
- D6 pad 1: /USB switch/SEL -> /Slide-SW/SEL
- D6 pad 2: /Slide-SW/SEL -> Net-(D6-Pad2)
- D7 pad 1: /USB switch/SEL -> /Slide-SW/SEL
- R31 pad 1: /GPIO_Expander/GPIO7 -> +3V3
- R8 pad 1: /USB switch/SEL -> /Slide-SW/SEL
- SW1 pad 3: /Slide-SW/SEL -> Net-(D6-Pad2)
Routing:
- net /USB switch/SEL: track 43.1 -> 0.00 mm, vias 3 -> 0
- net /Slide-SW/SEL: track 8.02 -> 47.2 mm, vias 0 -> 3
- net /UART_Programmer/~{DTR}: track 12.4 -> 28.2 mm, vias 2 -> 3
- net /UART_Programmer/~{RTS}: track 6.38 -> 21.8 mm, vias 0 -> 2
- net /ESP32-C6/UART0.TX: track 49.6 -> 59.0 mm
- net +3V3: track 244.9 -> 253.8 mm, vias 24 -> 29
- net /ESP32-C6/UART0.RX: track 49.5 -> 56.4 mm
- net /ESP32-C6/EN: track 50.4 -> 43.8 mm, vias 5 -> 6
- net /GPIO_Expander/GPIO7: track 5.36 -> 0.00 mm
- net /USBC_CONN/VBUS: track 33.8 -> 28.5 mm, vias 6 -> 7
- net /UART_Programmer/Prg.D+: track 6.47 -> 11.5 mm
- net /UART_Programmer/XI: track 8.02 -> 3.97 mm
- net Net-(D6-Pad2): track 0.00 -> 3.95 mm
- net /UART_Programmer/Prg.D-: track 7.00 -> 10.9 mm
- net Net-(Q2-B): track 7.56 -> 3.88 mm
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- added copper zone on B.Cu, net +3V3
- added copper zone on F.Cu, net +3V3
- added copper zone on F.Cu, net /USBC_CONN/VBUS
