File: MMS3/MMS3_ESP32-C6.kicad_sch (KiCad schematic)
At the start: 5 parts

Commit message: backup commit
Parts:
- added D7, D8: D, symbol Device:D
Connections:
- net Slide-SW/SEL: now also D8.2 (A)
- new net Select_GPIO: D7.2 (A)
- new net USB switch/SEL: D7.1 (K), D8.1 (K)
Other:
- sheet Input-Output renamed User IO
- sheet ESP32-C6 ports: added EN, IO9, UART0{UART}, USB{USB}; removed none
- sheet GPIO_Expander ports: added I2C{I2C}; removed 1wire_Uart
- sheet UART_Programmer ports: added EN, IO_9, Prg{UART}, Prg{USB}; removed none
- note added: "+Cstray"

Commit message: working commit
Changed lines of the file:
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@@
 	)
 	(bus_entry
+		(at 372.11 203.2)
+		(size 2.54 -2.54)
+		(stroke
+			(width 0)
+			(type default)
+		)
+	)
+	(bus_entry
+		(at 374.65 182.88)
+		(size -2.54 2.54)
+		(stroke
+			(width 0)
+			(type default)
+		)
+	)
+	(bus_entry
 		(at 339.09 200.66)
 		(size 2.54 2.54)
@@
 	)
 	(bus_entry
+		(at 374.65 203.2)
+		(size -2.54 2.54)
+		(stroke
+			(width 0)
+			(type default)
+		)
+	)
+	(bus_entry
+		(at 374.65 180.34)
+		(size -2.54 2.54)
+		(stroke
+			(width 0)
+			(type default)
+		)
+	)
+	(bus_entry
 		(at 339.09 203.2)
 		(size 2.54 2.54)
@@
 	(wire
 		(pts
-			(xy 364.49 205.74) (xy 341.63 205.74)
+			(xy 341.63 205.74) (xy 372.11 205.74)
 		)
 		(stroke
@@
 	(wire
 		(pts
-			(xy 364.49 203.2) (xy 341.63 203.2)
+			(xy 341.63 203.2) (xy 372.11 203.2)
 		)
 		(stroke
@@
 	(wire
 		(pts
-			(xy 364.49 182.88) (xy 341.63 182.88)
+			(xy 341.63 182.88) (xy 372.11 182.88)
 		)
 		(stroke
@@
 	(wire
 		(pts
-			(xy 364.49 185.42) (xy 341.63 185.42)
+			(xy 341.63 185.42) (xy 372.11 185.42)
 		)
 		(stroke
@@
 		)
 	)
+	(label "Altmode1"
+		(at 369.57 185.42 180)
+		(effects
+			(font
+				(size 1.27 1.27)
+			)
+			(justify right bottom)
+		)
+	)
 	(label "CAN2.TX"
 		(at 349.25 185.42 180)
@@
 		)
 	)
+	(label "Altmode3"
+		(at 369.57 205.74 180)
+		(effects
+			(font
+				(size 1.27 1.27)
+			)
+			(justify right bottom)
+		)
+	)
 	(label "CAN1{RX TX}"
 		(at 325.12 198.12 180)
@@
 		)
 	)
+	(label "Altmode2"
+		(at 369.57 182.88 180)
+		(effects
+			(font
+				(size 1.27 1.27)
+			)
+			(justify right bottom)
+		)
+	)
 	(label "RJ45_DWN_RX1"
 		(at 359.41 99.06 0)
@@
 		(effects
 			(font
+				(size 1.27 1.27)
+			)
+			(justify right bottom)
+		)
+	)
+	(label "Altmode4"
+		(at 369.57 203.2 180)
+		(effects
+			(font

Commit message: initial routing done
Parts:
- removed D7, D8: D, symbol Device:D
- added D6, D7: 1N5819WS, PCM_JLCPCB:D_SOD-323, symbol PCM_JLCPCB-Diodes:Schottky,1N5819WS
Connections:
- net Select_GPIO: now also D7.2
- net Slide-SW/SEL: now also D6.2
- net USB switch/SEL: now also D6.1, D7.1
Other:
- sheet GPIO_Expander ports: added GPIO[0..12], RJ45_DWN_RX1, RJ45_DWN_TX1, RJ45_UP_RX1, RJ45_UP_TX1, Select_GPIO; removed GPIO[0..11]
- sheet User IO ports: added GPIO[0..12]; removed GPIO[0..11], RJ45_DWN_RX1, RJ45_DWN_TX1, RJ45_UP_RX1, RJ45_UP_TX1

Commit message: routing done
Other:
- note removed: "+Cstray"
Changed lines of the file:
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@@
-		)
-	)
-	(text "+Cstray"
-		(exclude_from_sim no)
-		(at 166.37 74.93 0)
-		(effects
-			(font
-				(size 5.08 5.08)
-				(thickness 1.016)
-				(bold yes)
-				(color 255 0 255 1)
-			)
 		)
 	)
@@
 	(bus
 		(pts
-			(xy 374.65 123.19) (xy 374.65 229.87)
-		)
-		(stroke
-			(width 0)
-			(type default)
-		)
-	)
-	(bus
-		(pts
 			(xy 339.09 179.07) (xy 339.09 182.88)
 		)
@@
 		)
 		(stroke
+			(width 0)
+			(type default)
+		)
+	)
+	(bus
+		(pts
+			(xy 374.65 203.2) (xy 374.65 123.19)
+		)
+		(stroke

Commit message: eem, done?
Parts:
- removed D6: 1N5819WS, PCM_JLCPCB:D_SOD-323, symbol PCM_JLCPCB-Diodes:Schottky,1N5819WS
Connections:
- net USB switch/SEL is gone; now on net Slide-SW/SEL: D7.1
