File: MMS3/MMS3_ESP32-C6.kicad_sch (KiCad schematic)
At the start: 6 parts

Commit message: fixed swapped RX/TX & D+/D_
Parts:
- removed D5: SM4007PL, PCM_JLCPCB:D_SOD-123FL, symbol PCM_JLCPCB-Diodes:General,SM4007PL
- added D9: 1N5819WS, PCM_JLCPCB:D_SOD-323, symbol PCM_JLCPCB-Diodes:Schottky,1N5819WS
Connections:
- net +5V: now also D9.1
- net USB switch1/SEL: now also D9.2
