File: MMS3/Slide-SW.kicad_sch (KiCad schematic)
At the start: 3 parts, among them SW4 SK12D07VG5

Commit message: finished routing
Parts:
- D6: DNP_Basic (none) -> DNP; Manufacturer Hubei KENTO Elec -> (none)
- R31: DNP_Basic (none) -> DNP; Manufacturer UNI-ROYAL(Uniroyal Elec) -> (none)
- SW4: DNP_Basic (none) -> DNP; Manufacturer SHOU HAN(首韩) -> (none)
Connections:
- net GND: now also D6.1; no longer R31.2
- net SEL: now also R31.1; no longer D6.2
- new net: D6.2, R31.2
Other:
- title: MMS3 -> MMS3 MCU ESP32-C6
- moved on the sheet: D6, R31

Commit message: temp commit
Parts:
- renumbered D6 to D2, R31 to R11, SW4 to SW1
Changed lines of the file:
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@@
 		(dnp no)
 		(fields_autoplaced yes)
-		(property "Reference" "R31"
+		(property "Reference" "R11"
 			(at 130.81 102.8699 0)
 			(show_name no)
@@
 			(project "MMS3_ESP32-C6"
 				(path "/712cea22-140d-4c92-923f-f4998caf3ecd/5332ca3b-efcd-4d9b-b822-d9c330b0dec7"
-					(reference "R31")
+					(reference "R11")
 					(unit 1)
 				)
@@
 		(dnp no)
 		(fields_autoplaced yes)
-		(property "Reference" "D6"
+		(property "Reference" "D2"
 			(at 130.81 110.3946 0)
 			(show_name no)
@@
 			(project "MMS3_ESP32-C6"
 				(path "/712cea22-140d-4c92-923f-f4998caf3ecd/5332ca3b-efcd-4d9b-b822-d9c330b0dec7"
-					(reference "D6")
+					(reference "D2")
 					(unit 1)
 				)
@@
 		(dnp no)
 		(fields_autoplaced yes)
-		(property "Reference" "SW4"
+		(property "Reference" "SW1"
 			(at 97.4099 88.9 0)
 			(show_name no)
@@
 			(project "MMS3_ESP32-C6"
 				(path "/712cea22-140d-4c92-923f-f4998caf3ecd/5332ca3b-efcd-4d9b-b822-d9c330b0dec7"
-					(reference "SW4")
+					(reference "SW1")
 					(unit 1)
 				)

Commit message: eem, done?
Parts:
- added D6: 1N5819WS, PCM_JLCPCB:D_SOD-323, symbol PCM_JLCPCB-Diodes:Schottky,1N5819WS
Connections:
- net SEL: now also D6.1; no longer SW1.3
- new net: D6.2, SW1.3
Other:
- moved on the sheet: D2, R11
