File: MMS3/USB HUB.kicad_sch (KiCad schematic)
At the start: 17 parts, among them U302 CH334P, Y900 Crystal_GND24

Commit message: finished routing
Other:
- title: MMS3 -> MMS3 MCU ESP32-C6
Changed lines of the file:
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@@
 	(paper "A4")
 	(title_block
-		(title "MMS3")
+		(title "MMS3 MCU ESP32-C6")
 		(date "2026-04-03")
 		(rev "XA1")
 		(company "(c) Modular Mechanica")
-		(comment 1 "Artem Horiunov")
+		(comment 1 "Wojciech Szafrański ")
 		(comment 2 "DESIGNED IN POLAND")
 	)
@@
 		)
 		(instances
-			(project "MMS3"
+			(project "MMS3_ESP32-C6"
 				(path "/712cea22-140d-4c92-923f-f4998caf3ecd/6d97a548-c5fd-464f-b259-1eef25670dc7"
 					(reference "R20")
@@
 		)
 		(instances
-			(project "MMS3"
+			(project "MMS3_ESP32-C6"
 				(path "/712cea22-140d-4c92-923f-f4998caf3ecd/6d97a548-c5fd-464f-b259-1eef25670dc7"
 					(reference "D301")
@@
 		)
 		(instances
-			(project "MMS3"
+			(project "MMS3_ESP32-C6"
 				(path "/712cea22-140d-4c92-923f-f4998caf3ecd/6d97a548-c5fd-464f-b259-1eef25670dc7"
 					(reference "#PWR0329")
@@
 		)
 		(instances
-			(project "MMS3"
+			(project "MMS3_ESP32-C6"
 				(path "/712cea22-140d-4c92-923f-f4998caf3ecd/6d97a548-c5fd-464f-b259-1eef25670dc7"
 					(reference "#PWR0900")
@@
 		)
 		(instances
-			(project "MMS3"
+			(project "MMS3_ESP32-C6"
 				(path "/712cea22-140d-4c92-923f-f4998caf3ecd/6d97a548-c5fd-464f-b259-1eef25670dc7"
 					(reference "#PWR0328")
@@
 		)
 		(instances
-			(project "MMS3"
+			(project "MMS3_ESP32-C6"
 				(path "/712cea22-140d-4c92-923f-f4998caf3ecd/6d97a548-c5fd-464f-b259-1eef25670dc7"
 					(reference "R902")
@@
 		)
 		(instances
-			(project "MMS3"
+			(project "MMS3_ESP32-C6"
 				(path "/712cea22-140d-4c92-923f-f4998caf3ecd/6d97a548-c5fd-464f-b259-1eef25670dc7"
 					(reference "U302")
@@
 		)
 		(instances
-			(project "MMS3"
+			(project "MMS3_ESP32-C6"
 				(path "/712cea22-140d-4c92-923f-f4998caf3ecd/6d97a548-c5fd-464f-b259-1eef25670dc7"
 					(reference "R17")
@@
 		)
 		(instances
-			(project "MMS3"
+			(project "MMS3_ESP32-C6"
 				(path "/712cea22-140d-4c92-923f-f4998caf3ecd/6d97a548-c5fd-464f-b259-1eef25670dc7"
 					(reference "#PWR0901")
@@
 		)
 		(instances
-			(project "MMS3"
+			(project "MMS3_ESP32-C6"
 				(path "/712cea22-140d-4c92-923f-f4998caf3ecd/6d97a548-c5fd-464f-b259-1eef25670dc7"
 					(reference "#PWR0905")
@@
 		)
 		(instances
-			(project "MMS3"
+			(project "MMS3_ESP32-C6"
 				(path "/712cea22-140d-4c92-923f-f4998caf3ecd/6d97a548-c5fd-464f-b259-1eef25670dc7"
 					(reference "R308")
@@
 		)
 		(instances
-			(project "MMS3"
+			(project "MMS3_ESP32-C6"
 				(path "/712cea22-140d-4c92-923f-f4998caf3ecd/6d97a548-c5fd-464f-b259-1eef25670dc7"
 					(reference "R18")
@@
 		)
 		(instances
-			(project "MMS3"
+			(project "MMS3_ESP32-C6"
 				(path "/712cea22-140d-4c92-923f-f4998caf3ecd/6d97a548-c5fd-464f-b259-1eef25670dc7"
 					(reference "R903")
@@
 		)
 		(instances
-			(project "MMS3"
+			(project "MMS3_ESP32-C6"
 				(path "/712cea22-140d-4c92-923f-f4998caf3ecd/6d97a548-c5fd-464f-b259-1eef25670dc7"
 					(reference "C902")
@@
 		)
 		(instances
-			(project "MMS3"
+			(project "MMS3_ESP32-C6"
 				(path "/712cea22-140d-4c92-923f-f4998caf3ecd/6d97a548-c5fd-464f-b259-1eef25670dc7"
 					(reference "R19")
@@
 		)
 		(instances
-			(project "MMS3"
+			(project "MMS3_ESP32-C6"
 				(path "/712cea22-140d-4c92-923f-f4998caf3ecd/6d97a548-c5fd-464f-b259-1eef25670dc7"
 					(reference "#PWR0902")
@@
 		)
 		(instances
-			(project "MMS3"
+			(project "MMS3_ESP32-C6"
 				(path "/712cea22-140d-4c92-923f-f4998caf3ecd/6d97a548-c5fd-464f-b259-1eef25670dc7"
 					(reference "C900")
@@
 		)
 		(instances
-			(project "MMS3"
+			(project "MMS3_ESP32-C6"
 				(path "/712cea22-140d-4c92-923f-f4998caf3ecd/6d97a548-c5fd-464f-b259-1eef25670dc7"
 					(reference "C904")
@@
 		)
 		(instances
-			(project "MMS3"
+			(project "MMS3_ESP32-C6"
 				(path "/712cea22-140d-4c92-923f-f4998caf3ecd/6d97a548-c5fd-464f-b259-1eef25670dc7"
 					(reference "R906")
@@
 		)
 		(instances
-			(project "MMS3"
+			(project "MMS3_ESP32-C6"
 				(path "/712cea22-140d-4c92-923f-f4998caf3ecd/6d97a548-c5fd-464f-b259-1eef25670dc7"
 					(reference "R907")
@@
 		)
 		(instances
-			(project "MMS3"
+			(project "MMS3_ESP32-C6"
 				(path "/712cea22-140d-4c92-923f-f4998caf3ecd/6d97a548-c5fd-464f-b259-1eef25670dc7"
 					(reference "#PWR0904")
@@
 		)
 		(instances
-			(project "MMS3"
+			(project "MMS3_ESP32-C6"
 				(path "/712cea22-140d-4c92-923f-f4998caf3ecd/6d97a548-c5fd-464f-b259-1eef25670dc7"
 					(reference "R21")
@@
 		)
 		(instances
-			(project "MMS3"
+			(project "MMS3_ESP32-C6"
 				(path "/712cea22-140d-4c92-923f-f4998caf3ecd/6d97a548-c5fd-464f-b259-1eef25670dc7"
 					(reference "Y900")
@@
 		)
 		(instances
-			(project "MMS3"
+			(project "MMS3_ESP32-C6"
 				(path "/712cea22-140d-4c92-923f-f4998caf3ecd/6d97a548-c5fd-464f-b259-1eef25670dc7"
 					(reference "R16")

Commit message: temp commit
Other:
- note removed: "BM-probe bypass"
- note removed: "STM32 direct link"
Changed lines of the file:
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@@
 	)
 	(rectangle
-		(start 113.588 118.5959)
-		(end 133.908 122.4059)
-		(stroke
-			(width 0)
-			(type dash)
-		)
-		(fill
-			(type none)
-		)
-	)
-	(rectangle
-		(start 45.72 128.27)
-		(end 66.04 132.08)
-		(stroke
-			(width 0)
-			(type dash)
-		)
-		(fill
-			(type none)
-		)
-	)
-	(rectangle
 		(start 46.99 139.7)
 		(end 113.284 143.51)
@@
 	)
 	(rectangle
-		(start 204.9952 123.7234)
-		(end 225.3152 127.5334)
+		(start 155.7192 142.5194)
+		(end 176.0392 146.3294)
 		(stroke
 			(width 0)
@@
 		)
 	)
-	(text "BM-probe bypass"
-		(exclude_from_sim no)
-		(at 55.88 130.302 0)
-		(effects
-			(font
-				(size 1.27 1.27)
-			)
-		)
-	)
 	(text "Hipity hopity SI is now my property :)"
 		(exclude_from_sim no)
@@
 	(text "USB HUB BYPASS"
 		(exclude_from_sim no)
-		(at 214.376 125.984 0)
-		(effects
-			(font
-				(size 1.27 1.27)
-			)
-		)
-	)
-	(text "STM32 direct link"
-		(exclude_from_sim no)
-		(at 122.682 120.65 0)
+		(at 165.1 144.78 0)
 		(effects
 			(font
@@
 		)
 	)
-	(polyline
-		(pts
-			(xy 81.3 124.006) (xy 84.2791 124.058)
-		)
-		(stroke
-			(width 0)
-			(type default)
-		)
-	)
 	(bus
 		(pts
@@
 		)
 	)
-	(polyline
-		(pts
-			(xy 54.448 126.74) (xy 67.148 112.77)
-		)
-		(stroke
-			(width 0)
-			(type default)
-		)
-	)
 	(wire
 		(pts
@@
 		)
 	)
-	(polyline
-		(pts
-			(xy 81.8972 125.8374) (xy 84.2791 124.058)
-		)
-		(stroke
-			(width 0)
-			(type default)
-		)
-	)
 	(wire
 		(pts
@@
 		)
 	)
-	(polyline
-		(pts
-			(xy 64.1489 114.442) (xy 67.148 112.77)
-		)
-		(stroke
-			(width 0)
-			(type default)
-		)
-	)
 	(wire
 		(pts
@@
 	(polyline
 		(pts
-			(xy 196.85 118.11) (xy 199.3533 119.041)
+			(xy 147.574 136.906) (xy 150.0773 137.837)
 		)
 		(stroke
@@
 		)
 	)
-	(polyline
-		(pts
-			(xy 66.04 115.57) (xy 67.148 112.77)
-		)
-		(stroke
-			(width 0)
-			(type default)
-		)
-	)
 	(wire
 		(pts
@@
 	(polyline
 		(pts
-			(xy 196.85 118.11) (xy 197.8327 120.064)
+			(xy 147.574 136.906) (xy 148.5567 138.86)
 		)
 		(stroke
@@
 	(polyline
 		(pts
-			(xy 196.85 118.11) (xy 204.47 124.46)
+			(xy 147.574 136.906) (xy 155.194 143.256)
 		)
 		(stroke
@@
 		)
 	)
-	(polyline
-		(pts
-			(xy 113.03 120.65) (xy 102.87 114.3)
-		)
-		(stroke
-			(width 0)
-			(type default)
-		)
-	)
 	(wire
 		(pts
@@
 		)
 	)
-	(polyline
-		(pts
-			(xy 102.87 114.3) (xy 105.8006 115.1836)
-		)
-		(stroke
-			(width 0)
-			(type default)
-		)
-	)
 	(wire
 		(pts
@@
 		)
 	)
-	(polyline
-		(pts
-			(xy 102.87 114.3) (xy 104.2479 116.7363)
-		)
-		(stroke
-			(width 0)
-			(type default)
-		)
-	)
 	(bus
 		(pts
@@
 		)
 	)
-	(polyline
-		(pts
-			(xy 67.31 128.27) (xy 84.2791 124.058)
-		)
-		(stroke
-			(width 0)
-			(type default)
-		)
-	)
 	(wire
 		(pts
@@
 		(instances
 			(project "MMS3_ESP32-C6"
-				(path "/712cea22-140d-4c92-923f-f4998caf3ecd/6d97a548-c5fd-464f-b259-1eef25670dc7"
+				(path "/712cea22-140d-4c92-923f-f4998caf3ecd/49d312a8-5b35-4365-b1f6-aa64c95e454a"
 					(reference "R20")
 					(unit 1)
@@
 		(instances
 			(project "MMS3_ESP32-C6"
-				(path "/712cea22-140d-4c92-923f-f4998caf3ecd/6d97a548-c5fd-464f-b259-1eef25670dc7"
+				(path "/712cea22-140d-4c92-923f-f4998caf3ecd/49d312a8-5b35-4365-b1f6-aa64c95e454a"
 					(reference "D301")
 					(unit 1)
@@
 		(instances
 			(project "MMS3_ESP32-C6"
-				(path "/712cea22-140d-4c92-923f-f4998caf3ecd/6d97a548-c5fd-464f-b259-1eef25670dc7"
+				(path "/712cea22-140d-4c92-923f-f4998caf3ecd/49d312a8-5b35-4365-b1f6-aa64c95e454a"
 					(reference "#PWR0329")
 					(unit 1)
@@
 		(instances
 			(project "MMS3_ESP32-C6"
-				(path "/712cea22-140d-4c92-923f-f4998caf3ecd/6d97a548-c5fd-464f-b259-1eef25670dc7"
+				(path "/712cea22-140d-4c92-923f-f4998caf3ecd/49d312a8-5b35-4365-b1f6-aa64c95e454a"
 					(reference "#PWR0900")
 					(unit 1)
@@
 		(instances
 			(project "MMS3_ESP32-C6"
-				(path "/712cea22-140d-4c92-923f-f4998caf3ecd/6d97a548-c5fd-464f-b259-1eef25670dc7"
+				(path "/712cea22-140d-4c92-923f-f4998caf3ecd/49d312a8-5b35-4365-b1f6-aa64c95e454a"
 					(reference "#PWR0328")
 					(unit 1)
@@
 		(instances
 			(project "MMS3_ESP32-C6"
-				(path "/712cea22-140d-4c92-923f-f4998caf3ecd/6d97a548-c5fd-464f-b259-1eef25670dc7"
+				(path "/712cea22-140d-4c92-923f-f4998caf3ecd/49d312a8-5b35-4365-b1f6-aa64c95e454a"
 					(reference "R902")
 					(unit 1)
@@
 		(instances
 			(project "MMS3_ESP32-C6"
-				(path "/712cea22-140d-4c92-923f-f4998caf3ecd/6d97a548-c5fd-464f-b259-1eef25670dc7"
+				(path "/712cea22-140d-4c92-923f-f4998caf3ecd/49d312a8-5b35-4365-b1f6-aa64c95e454a"
 					(reference "U302")
 					(unit 1)
@@
 		(instances
 			(project "MMS3_ESP32-C6"
-				(path "/712cea22-140d-4c92-923f-f4998caf3ecd/6d97a548-c5fd-464f-b259-1eef25670dc7"
+				(path "/712cea22-140d-4c92-923f-f4998caf3ecd/49d312a8-5b35-4365-b1f6-aa64c95e454a"
 					(reference "R17")
 					(unit 1)
@@
 		(instances
 			(project "MMS3_ESP32-C6"
-				(path "/712cea22-140d-4c92-923f-f4998caf3ecd/6d97a548-c5fd-464f-b259-1eef25670dc7"
+				(path "/712cea22-140d-4c92-923f-f4998caf3ecd/49d312a8-5b35-4365-b1f6-aa64c95e454a"
 					(reference "#PWR0901")
 					(unit 1)
@@
 		(instances
 			(project "MMS3_ESP32-C6"
-				(path "/712cea22-140d-4c92-923f-f4998caf3ecd/6d97a548-c5fd-464f-b259-1eef25670dc7"
+				(path "/712cea22-140d-4c92-923f-f4998caf3ecd/49d312a8-5b35-4365-b1f6-aa64c95e454a"
 					(reference "#PWR0905")
 					(unit 1)
@@
 		(instances
 			(project "MMS3_ESP32-C6"
-				(path "/712cea22-140d-4c92-923f-f4998caf3ecd/6d97a548-c5fd-464f-b259-1eef25670dc7"
+				(path "/712cea22-140d-4c92-923f-f4998caf3ecd/49d312a8-5b35-4365-b1f6-aa64c95e454a"
 					(reference "R308")
 					(unit 1)
@@
 		(instances
 			(project "MMS3_ESP32-C6"
-				(path "/712cea22-140d-4c92-923f-f4998caf3ecd/6d97a548-c5fd-464f-b259-1eef25670dc7"
+				(path "/712cea22-140d-4c92-923f-f4998caf3ecd/49d312a8-5b35-4365-b1f6-aa64c95e454a"
 					(reference "R18")
 					(unit 1)
@@
 		(instances
 			(project "MMS3_ESP32-C6"
-				(path "/712cea22-140d-4c92-923f-f4998caf3ecd/6d97a548-c5fd-464f-b259-1eef25670dc7"
+				(path "/712cea22-140d-4c92-923f-f4998caf3ecd/49d312a8-5b35-4365-b1f6-aa64c95e454a"
 					(reference "R903")
 					(unit 1)
@@
 		(instances
 			(project "MMS3_ESP32-C6"
-				(path "/712cea22-140d-4c92-923f-f4998caf3ecd/6d97a548-c5fd-464f-b259-1eef25670dc7"
+				(path "/712cea22-140d-4c92-923f-f4998caf3ecd/49d312a8-5b35-4365-b1f6-aa64c95e454a"
 					(reference "C902")
 					(unit 1)
@@
 		(instances
 			(project "MMS3_ESP32-C6"
-				(path "/712cea22-140d-4c92-923f-f4998caf3ecd/6d97a548-c5fd-464f-b259-1eef25670dc7"
+				(path "/712cea22-140d-4c92-923f-f4998caf3ecd/49d312a8-5b35-4365-b1f6-aa64c95e454a"
 					(reference "R19")
 					(unit 1)
@@
 		(instances
 			(project "MMS3_ESP32-C6"
-				(path "/712cea22-140d-4c92-923f-f4998caf3ecd/6d97a548-c5fd-464f-b259-1eef25670dc7"
+				(path "/712cea22-140d-4c92-923f-f4998caf3ecd/49d312a8-5b35-4365-b1f6-aa64c95e454a"
 					(reference "#PWR0902")
 					(unit 1)
@@
 		(instances
 			(project "MMS3_ESP32-C6"
-				(path "/712cea22-140d-4c92-923f-f4998caf3ecd/6d97a548-c5fd-464f-b259-1eef25670dc7"
+				(path "/712cea22-140d-4c92-923f-f4998caf3ecd/49d312a8-5b35-4365-b1f6-aa64c95e454a"
 					(reference "C900")
 					(unit 1)
@@
 		(instances
 			(project "MMS3_ESP32-C6"
-				(path "/712cea22-140d-4c92-923f-f4998caf3ecd/6d97a548-c5fd-464f-b259-1eef25670dc7"
+				(path "/712cea22-140d-4c92-923f-f4998caf3ecd/49d312a8-5b35-4365-b1f6-aa64c95e454a"
 					(reference "C904")
 					(unit 1)
@@
 		(instances
 			(project "MMS3_ESP32-C6"
-				(path "/712cea22-140d-4c92-923f-f4998caf3ecd/6d97a548-c5fd-464f-b259-1eef25670dc7"
+				(path "/712cea22-140d-4c92-923f-f4998caf3ecd/49d312a8-5b35-4365-b1f6-aa64c95e454a"
 					(reference "R906")
 					(unit 1)
@@
 		(instances
 			(project "MMS3_ESP32-C6"
-				(path "/712cea22-140d-4c92-923f-f4998caf3ecd/6d97a548-c5fd-464f-b259-1eef25670dc7"
+				(path "/712cea22-140d-4c92-923f-f4998caf3ecd/49d312a8-5b35-4365-b1f6-aa64c95e454a"
 					(reference "R907")
 					(unit 1)
@@
 		(instances
 			(project "MMS3_ESP32-C6"
-				(path "/712cea22-140d-4c92-923f-f4998caf3ecd/6d97a548-c5fd-464f-b259-1eef25670dc7"
+				(path "/712cea22-140d-4c92-923f-f4998caf3ecd/49d312a8-5b35-4365-b1f6-aa64c95e454a"
 					(reference "#PWR0904")
 					(unit 1)
@@
 		(instances
 			(project "MMS3_ESP32-C6"
-				(path "/712cea22-140d-4c92-923f-f4998caf3ecd/6d97a548-c5fd-464f-b259-1eef25670dc7"
+				(path "/712cea22-140d-4c92-923f-f4998caf3ecd/49d312a8-5b35-4365-b1f6-aa64c95e454a"
 					(reference "R21")
 					(unit 1)
@@
 		(instances
 			(project "MMS3_ESP32-C6"
-				(path "/712cea22-140d-4c92-923f-f4998caf3ecd/6d97a548-c5fd-464f-b259-1eef25670dc7"
+				(path "/712cea22-140d-4c92-923f-f4998caf3ecd/49d312a8-5b35-4365-b1f6-aa64c95e454a"
 					(reference "Y900")
 					(unit 1)
@@
 		(instances
 			(project "MMS3_ESP32-C6"
-				(path "/712cea22-140d-4c92-923f-f4998caf3ecd/6d97a548-c5fd-464f-b259-1eef25670dc7"
+				(path "/712cea22-140d-4c92-923f-f4998caf3ecd/49d312a8-5b35-4365-b1f6-aa64c95e454a"
 					(reference "R16")
 					(unit 1)

Commit message: initial routing done
Parts:
- removed R21: 22Ω, PCM_JLCPCB:R_0402, symbol PCM_JLCPCB-Resistors:0402,22Ω
Connections:
- net USBBYP.D+ is gone; now on net USBOUT1.D+: R18.1

Commit message: eem, done?
Parts:
- U302: LCSC (none) -> C5373042
