File: MMS3/USB switch.kicad_sch (KiCad schematic)
At the start: 5 parts, among them U802 FSUSB42UMX

Commit message: finished routing
Parts:
- C312: renamed from C313; DNP_Basic (none) -> DNP; Manufacturer Samsung Electro-Mechanics -> (none)
- R802: renamed from R805; DNP_Basic (none) -> DNP; Manufacturer UNI-ROYAL(Uniroyal Elec) -> (none)
- R803: renamed from R806; DNP_Basic (none) -> DNP; Manufacturer UNI-ROYAL(Uniroyal Elec) -> (none)
- R804: renamed from R807; DNP_Basic (none) -> DNP; Manufacturer UNI-ROYAL(Uniroyal Elec) -> (none)
- U801: renamed from U802; DNP_Basic (none) -> DNP
Connections:
- net USB_OUT1.D+: now also U801.5 (HSD1+); no longer U801.7 (HSD2+)
- net USB_OUT1.D-: now also U801.4 (HSD1-); no longer U801.6 (HSD2-)
- net USB_OUT2.D+: now also U801.7 (HSD2+); no longer U801.5 (HSD1+)
- net USB_OUT2.D-: now also U801.6 (HSD2-); no longer U801.4 (HSD1-)
Other:
- title: MMS3 -> MMS3 MCU ESP32-C6

Commit message: temp commit
Parts:
- renumbered C312 to C5, R804 to R10, R802 to R8, R803 to R9, U801 to U3
Changed lines of the file:
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@@
 		(dnp no)
 		(fields_autoplaced yes)
-		(property "Reference" "C312"
+		(property "Reference" "C5"
 			(at 151.13 82.5499 0)
 			(show_name no)
@@
 			(project "MMS3_ESP32-C6"
 				(path "/712cea22-140d-4c92-923f-f4998caf3ecd/588e5e8a-0269-4161-b9f0-fd5ae057e0d0"
-					(reference "C312")
+					(reference "C5")
 					(unit 1)
 				)
 				(path "/712cea22-140d-4c92-923f-f4998caf3ecd/d394fa85-d1a1-4f94-8f54-7ea4e8d94b3a"
-					(reference "C313")
+					(reference "C8")
 					(unit 1)
 				)
@@
 		(dnp no)
 		(fields_autoplaced yes)
-		(property "Reference" "U801"
+		(property "Reference" "U3"
 			(at 125.73 80.01 0)
 			(show_name no)
@@
 			(project "MMS3_ESP32-C6"
 				(path "/712cea22-140d-4c92-923f-f4998caf3ecd/588e5e8a-0269-4161-b9f0-fd5ae057e0d0"
-					(reference "U801")
+					(reference "U3")
 					(unit 1)
 				)
 				(path "/712cea22-140d-4c92-923f-f4998caf3ecd/d394fa85-d1a1-4f94-8f54-7ea4e8d94b3a"
-					(reference "U802")
+					(reference "U7")
 					(unit 1)
 				)
@@
 		(in_pos_files yes)
 		(dnp no)
-		(property "Reference" "R804"
+		(property "Reference" "R10"
 			(at 109.22 119.38 0)
 			(show_name no)
@@
 			(project "MMS3_ESP32-C6"
 				(path "/712cea22-140d-4c92-923f-f4998caf3ecd/588e5e8a-0269-4161-b9f0-fd5ae057e0d0"
-					(reference "R804")
+					(reference "R10")
 					(unit 1)
 				)
 				(path "/712cea22-140d-4c92-923f-f4998caf3ecd/d394fa85-d1a1-4f94-8f54-7ea4e8d94b3a"
-					(reference "R807")
+					(reference "R15")
 					(unit 1)
 				)
@@
 		(in_pos_files yes)
 		(dnp no)
-		(property "Reference" "R802"
+		(property "Reference" "R8"
 			(at 93.98 110.744 90)
 			(show_name no)
@@
 			(project "MMS3_ESP32-C6"
 				(path "/712cea22-140d-4c92-923f-f4998caf3ecd/588e5e8a-0269-4161-b9f0-fd5ae057e0d0"
-					(reference "R802")
+					(reference "R8")
 					(unit 1)
 				)
 				(path "/712cea22-140d-4c92-923f-f4998caf3ecd/d394fa85-d1a1-4f94-8f54-7ea4e8d94b3a"
-					(reference "R805")
+					(reference "R13")
 					(unit 1)
 				)
@@
 		(in_pos_files yes)
 		(dnp no)
-		(property "Reference" "R803"
+		(property "Reference" "R9"
 			(at 100.33 119.38 0)
 			(show_name no)
@@
 			(project "MMS3_ESP32-C6"
 				(path "/712cea22-140d-4c92-923f-f4998caf3ecd/588e5e8a-0269-4161-b9f0-fd5ae057e0d0"
-					(reference "R803")
+					(reference "R9")
 					(unit 1)
 				)
 				(path "/712cea22-140d-4c92-923f-f4998caf3ecd/d394fa85-d1a1-4f94-8f54-7ea4e8d94b3a"
-					(reference "R806")
+					(reference "R14")
 					(unit 1)
 				)
