File: MMS3/USBC_CONN.kicad_sch (KiCad schematic)
At the start: 7 parts, among them J800 USB_C_Receptacle_USB2.0_16P, U401 TPD2EUSB30DRTR-TP

Commit message: finished routing
Parts:
- removed C7: 10nF, PCM_JLCPCB:C_0402, symbol PCM_JLCPCB-Capacitors:0402,10nF
- removed C800: 100nF, PCM_JLCPCB:C_0402, symbol PCM_JLCPCB-Capacitors:0402,100nF,(2)
- removed R7: 33kΩ, PCM_JLCPCB:R_0402, symbol PCM_JLCPCB-Resistors:0402,33kΩ
- removed R8, R9: 5.1kΩ, PCM_JLCPCB:R_0402, symbol PCM_JLCPCB-Resistors:0402,5.1kΩ
- added C3: 10nF, PCM_JLCPCB:C_0603, symbol PCM_JLCPCB-Capacitors:0603,10nF
- added C4: 100nF, PCM_JLCPCB:C_0603, symbol PCM_JLCPCB-Capacitors:0603,100nF
- added R10: 33kΩ, PCM_JLCPCB:R_0603, symbol PCM_JLCPCB-Resistors:0603,33kΩ
- added R7, R8: 5.1kΩ, PCM_JLCPCB:R_0603, symbol PCM_JLCPCB-Resistors:0603,5.1kΩ
Connections:
- net CC1: now also R7.1
- net CC2: now also R8.1
- net GND: now also C3.2, C4.2, R10.2, R7.2, R8.2
- net USBC_CONN.D+: now also U401.2; no longer U401.1
- net USBC_CONN.D-: now also U401.1; no longer U401.2
- net VBUS: now also C4.1
- net at J800.SH (SHIELD): now also C3.1, R10.1
Other:
- title: MMS3 -> MMS3 MCU ESP32-C6

Commit message: temp commit
Parts:
- renumbered C3 to C14, C4 to C15, J800 to J4, R10 to R27, R8 to R28, R7 to R29, U401 to U9
Changed lines of the file:
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@@
 		(in_pos_files yes)
 		(dnp no)
-		(property "Reference" "R8"
+		(property "Reference" "R28"
 			(at 125.984 103.124 90)
 			(show_name no)
@@
 			(project "MMS3_ESP32-C6"
 				(path "/712cea22-140d-4c92-923f-f4998caf3ecd/6293ce90-9b00-41f8-95cd-8a2592163f0a"
-					(reference "R8")
+					(reference "R28")
 					(unit 1)
 				)
@@
 		(dnp no)
 		(fields_autoplaced yes)
-		(property "Reference" "C4"
+		(property "Reference" "C15"
 			(at 140.97 74.9299 0)
 			(show_name no)
@@
 			(project "MMS3_ESP32-C6"
 				(path "/712cea22-140d-4c92-923f-f4998caf3ecd/6293ce90-9b00-41f8-95cd-8a2592163f0a"
-					(reference "C4")
+					(reference "C15")
 					(unit 1)
 				)
@@
 		(in_pos_files yes)
 		(dnp no)
-		(property "Reference" "R7"
+		(property "Reference" "R29"
 			(at 134.366 102.87 90)
 			(show_name no)
@@
 			(project "MMS3_ESP32-C6"
 				(path "/712cea22-140d-4c92-923f-f4998caf3ecd/6293ce90-9b00-41f8-95cd-8a2592163f0a"
-					(reference "R7")
+					(reference "R29")
 					(unit 1)
 				)
@@
 		(in_pos_files yes)
 		(dnp no)
-		(property "Reference" "C3"
+		(property "Reference" "C14"
 			(at 102.87 125.73 90)
 			(show_name no)
@@
 			(project "MMS3_ESP32-C6"
 				(path "/712cea22-140d-4c92-923f-f4998caf3ecd/6293ce90-9b00-41f8-95cd-8a2592163f0a"
-					(reference "C3")
+					(reference "C14")
 					(unit 1)
 				)
@@
 		(dnp no)
 		(fields_autoplaced yes)
-		(property "Reference" "J800"
+		(property "Reference" "J4"
 			(at 100.33 66.04 0)
 			(show_name no)
@@
 			(project "MMS3_ESP32-C6"
 				(path "/712cea22-140d-4c92-923f-f4998caf3ecd/6293ce90-9b00-41f8-95cd-8a2592163f0a"
-					(reference "J800")
+					(reference "J4")
 					(unit 1)
 				)
@@
 		(in_pos_files yes)
 		(dnp no)
-		(property "Reference" "R10"
+		(property "Reference" "R27"
 			(at 94.996 126.238 90)
 			(show_name no)
@@
 			(project "MMS3_ESP32-C6"
 				(path "/712cea22-140d-4c92-923f-f4998caf3ecd/6293ce90-9b00-41f8-95cd-8a2592163f0a"
-					(reference "R10")
+					(reference "R27")
 					(unit 1)
 				)
@@
 		(dnp no)
 		(fields_autoplaced yes)
-		(property "Reference" "U401"
+		(property "Reference" "U9"
 			(at 157.48 100.3299 0)
 			(show_name no)
@@
 			(project "MMS3_ESP32-C6"
 				(path "/712cea22-140d-4c92-923f-f4998caf3ecd/6293ce90-9b00-41f8-95cd-8a2592163f0a"
-					(reference "U401")
+					(reference "U9")
 					(unit 1)
 				)

Commit message: backup commit
Parts:
- removed C14: 10nF, PCM_JLCPCB:C_0603, symbol PCM_JLCPCB-Capacitors:0603,10nF
- removed C15: 100nF, PCM_JLCPCB:C_0603, symbol PCM_JLCPCB-Capacitors:0603,100nF
- removed R27: 33kΩ, PCM_JLCPCB:R_0603, symbol PCM_JLCPCB-Resistors:0603,33kΩ
- removed R28, R29: 5.1kΩ, PCM_JLCPCB:R_0603, symbol PCM_JLCPCB-Resistors:0603,5.1kΩ
- added C12: 100nF, PCM_JLCPCB:C_0402, symbol PCM_JLCPCB-Capacitors:0402,100nF
- added C13: 10nF, PCM_JLCPCB:C_0402, symbol PCM_JLCPCB-Capacitors:0402,10nF
- added R25, R26: 5.1kΩ, PCM_JLCPCB:R_0402, symbol PCM_JLCPCB-Resistors:0402,5.1kΩ
- added R27: 33kΩ, PCM_JLCPCB:R_0402, symbol PCM_JLCPCB-Resistors:0402,33kΩ
Connections:
- net CC1: now also R25.1
- net CC2: now also R26.1
- net GND: now also C12.2, C13.2, R25.2, R26.2, R27.2
- net VBUS: now also C12.1
- net at J4.SH (SHIELD): now also C13.1, R27.1
