File: MMS3/ESP32-C6_chip.kicad_sch (KiCad schematic)
At the start: 33 parts, among them J5 Conn_Coaxial, U11 ESP32-C6_C5364646, U12 W25Q128, X2 40MHz, 15pF

Commit message: backup commit
Parts:
- removed C19, C22, C24: C, symbol Device:C
- removed C48: 1uF, PCM_JLCPCB:C_0402, symbol PCM_JLCPCB-Capacitors:0402,1uF
- removed L3: L, symbol Device:L
- removed L5: 24 nH???, symbol Device:L
- removed U12: W25Q128, PCM_JLCPCB:SOIC-8_L5.3-W5.3-P1.27-LS8.0-BL, symbol PCM_JLCPCB-Memory:16MByte, SPI
- added C19: 1uF, PCM_JLCPCB:C_0402, symbol PCM_JLCPCB-Capacitors:0402,1uF
- added C22: 1.5pF, PCM_JLCPCB:C_0402, symbol PCM_JLCPCB-Capacitors:0402,1.5pF
- added C52, C53: 100nF, PCM_JLCPCB:C_0402, symbol PCM_JLCPCB-Capacitors:0402,100nF
- added C57, C58: 30pF, PCM_JLCPCB:C_0402, symbol PCM_JLCPCB-Capacitors:0402,30pF
- added C59: 10uF, PCM_JLCPCB:C_0402, symbol PCM_JLCPCB-Capacitors:0402,10uF
- added L5: 3.9nH,300mA, PCM_JLCPCB:L_0402, symbol PCM_JLCPCB-Inductors:3.9nH,300mA
- added R22: 0Ω, PCM_JLCPCB:R_0402, symbol PCM_JLCPCB-Resistors:0402,0Ω
- added R52, R53, R54, R55, R56: 10kΩ, PCM_JLCPCB:R_0402, symbol PCM_JLCPCB-Resistors:0402,10kΩ
- added SW3, SW4: TC-6615Z-12.5-260, Tact-sw:SW-TH_4P-L7.3-TC-6615Z-12.5-260, symbol Tact-sw:TC-6615Z-12.5-260
- added U14: XT25F128FWOIGT-W, SPI_flash:WSON-8_L6.0-W5.0-P1.27-BL-EP, symbol SPI_flash:XT25F128FWOIGT-W
- C17, C18: value C -> DNI
- L2: value L -> DNI
Connections:
- net GPIO0 is gone; now on net Chainbus_addr2: U11.6 (XTAL_32K_P)
- net GPIO1 is gone; now on net Chainbus_addr1: U11.7 (XTAL_32K_N)
- net GPIO10 is gone; now on net Chainbus_addr7: U11.16 (GPIO10)
- net GPIO11 is gone; now on net Chainbus_addr6: U11.17 (GPIO11)
- net GPIO15 is gone; now on net Altmode3: U11.27 (GPIO15)
- net GPIO18 is gone; now on net Chainbus.SCK: U11.31 (SDIO_CMD)
- net GPIO19 is gone; now on net Chainbus.MOSI: U11.32 (SDIO_CLK)
- net GPIO2 is gone; now on net Chainbus_addr3: U11.8 (GPIO2)
- net GPIO20 is gone; now on net Chainbus.MISO: U11.33 (SDIO_DATA0)
- net GPIO21 is gone; now on net Altmode1: U11.34 (SDIO_DATA1)
- net GPIO22 is gone; now on net Altmode2: U11.35 (SDIO_DATA2)
- net GPIO23 is gone; now on net Chainbus.CS: U11.36 (SDIO_DATA3)
- net GPIO3 is gone; now on net Chainbus_addr4: U11.9 (GPIO3)
- net GPIO4 is gone; now on net Chainbus.RX: U11.10 (MTMS)
- net GPIO5 is gone; now on net Chainbus.TX: U11.11 (MTDI)
- net GPIO6 is gone; now on net Chainbus.SDA: U11.12 (MTCK)
- net GPIO7 is gone; now on net Chainbus.SCL: U11.13 (MTDO)
- net GPIO8 is gone; now on net Chainbus_addr5: U11.14 (GPIO8)
- net +3V3: now also C37.1, U11.28 (VDDPST2), U11.5 (VDDPST1), C52.1, C53.1, C59.1, R52.2, R53.2, R54.2, R55.1, R56.1, U14.8 (VCC); no longer C36.1
- net Altmode4: now also U11.23 (VDD_SPI)
- net Chainbus.RX: now also R55.2
- net Chainbus.TX: now also R56.2
- net Chainbus_addr5: now also R54.1
- net EN: now also C19.1, R53.1, SW3.1 (A)
- net GND: now also C19.2, C52.2, C53.2, C57.2, C58.2, C59.2, L5.2, SW3.2 (B), SW3.3 (C), SW3.4 (D), SW4.2 (B), SW4.3 (C), SW4.4 (D), U14.4 (VSS), U14.9 (EP)
- net SPICLK: now also U14.6 (SCLK)
- net SPICS0: now also U14.1 (~{CS})
- net SPID: now also U14.5 (SI(IO0))
- net SPIHD: now also U14.7 (HOLD#(IO3))
- net SPIQ: now also U14.2 (SO(IO1))
- net SPIWP: now also U14.3 (WP#(IO2))
- net XTAL_N: now also C57.1
- net XTAL_P: now also R22.2
- net ESP_SPICS0: now reaches R47.1, U11.20 (SPICS0)
- net ESP_TX: now reaches R49.2, U11.29 (U0TXD)
- net VCC_RF: now reaches C25.1, FB1.1, U11.2 (VDDA3P3), U11.3 (VDDA3P3)
- net VCC_RF: now also C36.1
- net ESP_SPIQ: now reaches R44.1, U11.21 (SPIQ)
- net ESP_SPIWP: now reaches R43.1, U11.22 (SPIWP)
- net ESP_SPIHD: now reaches R45.1, U11.24 (SPIHD)
- net ESP_CSPICLK: now reaches R48.1, U11.25 (SPICLK)
- net ESP_SPID: now reaches R46.1, U11.26 (SPID)
- net at C18.1, L2.2: now also C22.1
- net at C20.1, L4.1: now also C22.2, L5.1
- net XTAL_P.: now reaches X2.1 (OSC)
- net XTAL_P.: now also C58.1, R22.1
- net GPIO9 renamed IO9
- net IO9: now also R52.1, SW4.1 (A)
- removed net VDD_SPI: C37.1, U11.23 (VDD_SPI)
- no-connect marks 2 -> 12
Other:
- note added: "+Cstray"
- note added: "Boot0"
- note added: "Boot1"
- note added: "Chainbus Address"
- note added: "Chainbus Altmode"
- note added: "Chainbus I2C"
- note added: "Chainbus SPI"
- note added: "Chainbus UART"
- note added: "EN (~{RST})"
- note added: "ESD"
- note added: "ESD on PSU"
- note added: "L Value"
- note added: "MTDI"
- note added: "MTMS"
- note added: "Pinout"
- note added: "SDIO edges"
- note added: "STRAPPING PINS GPIO8, GPIO9, GPIO15, MTMS, and MTDI are strapping pins. GPIO4 GPIO5 are MTMS MTDI"
- note added: "Should be 24nH"
- note added: "Strapping Pins"
- note added: "Value"
- note added: "add a stub to ground pad"
- note removed: "AltMode pins"
- note removed: "ChainBus addressing"
- note removed: "ChainBus protocols"
- note removed: "GOOD?"
- moved on the sheet: C25, C26, C27, C28, C29, C37, FB1, R43, R44, R45, R46, R47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

Commit message: working commit
Parts:
- removed C17, C18: DNI, symbol Device:C
- removed C20, C21: C, symbol Device:C
- removed C36: 10uF, PCM_JLCPCB:C_0402, symbol PCM_JLCPCB-Capacitors:0402,10uF
- removed L2: DNI, symbol Device:L
- removed L4: L, symbol Device:L
- removed R22: 0Ω, PCM_JLCPCB:R_0402, symbol PCM_JLCPCB-Resistors:0402,0Ω
- removed U14: XT25F128FWOIGT-W, SPI_flash:WSON-8_L6.0-W5.0-P1.27-BL-EP, symbol SPI_flash:XT25F128FWOIGT-W
- added C17: 2.2pF, PCM_JLCPCB:C_0402, symbol PCM_JLCPCB-Capacitors:0402,2.2pF
- added C18: 3.3pF, PCM_JLCPCB:C_0402, symbol PCM_JLCPCB-Capacitors:0402,3.3pF
- added L2: 15nH,300mA, PCM_JLCPCB:L_0402, symbol PCM_JLCPCB-Inductors:15nH,300mA
- added L3: 2n, PCM_JLCPCB:C_0402, symbol Device:L
- added R42, R57, R58: 0Ω, PCM_JLCPCB:R_0402, symbol PCM_JLCPCB-Resistors:0402,0Ω
- added U8: ZD25Q128CSIGT, spi_flash:SOP-8_L5.3-W5.3-P1.27-LS7.9-BL, symbol spi_flash:ZD25Q128CSIGT
Connections:
- net +3V3: now also U8.8 (VCC)
- net ANT: now also C18.1, L3.1
- net Altmode1: now also U11.35 (SDIO_DATA2); no longer U11.34 (SDIO_DATA1)
- net Altmode2: now also U11.34 (SDIO_DATA1); no longer U11.35 (SDIO_DATA2)
- net GND: now also C17.2, C18.2, R57.1, R58.1, U8.4 (VSS)
- net SPICLK: now also U8.6 (SCLK)
- net SPICS0: now also U8.1 (~{CS})
- net SPID: now also U8.5 (SI(IO0))
- net SPIHD: now also U8.7 (~{HOLD}/RESET#(IO3))
- net SPIQ: now also U8.2 (SO(IO1))
- net SPIWP: now also U8.3 (WP#(IO2))
- net XTAL_P: now also L2.2
- net XTAL_P.: now also L2.1
- net More_RF: now reaches C22.2, L5.1
- net More_RF: now also R42.1, R57.2
- net RF: now reaches C22.1
- net RF: now also C17.1, L3.2
- net ANT_CN: now reaches J5.1 (In)
- net ANT_CN: now also R42.2, R58.2
Other:
- note added: "VSWR = 1.15"
- note added: "assuming Z = 32 + j5"
- note removed: "Value"
- moved on the sheet: C37

Commit message: initial routing done
Parts:
- removed SW4: TC-6615Z-12.5-260, Tact-sw:SW-TH_4P-L7.3-TC-6615Z-12.5-260, symbol Tact-sw:TC-6615Z-12.5-260
- added R59, R60: 10kΩ, PCM_JLCPCB:R_0402, symbol PCM_JLCPCB-Resistors:0402,10kΩ
Connections:
- net Chainbus_addr7 is gone; now on net Chainbus_addr6: U11.16 (GPIO10)
- net +3V3: now also R59.2, R60.2
- net Chainbus.SCL: now also R59.1
- net Chainbus.SDA: now also R60.1
- net Chainbus_addr1: now also U11.6 (XTAL_32K_P); no longer U11.7 (XTAL_32K_N)
- net Chainbus_addr2: now also U11.7 (XTAL_32K_N); no longer U11.6 (XTAL_32K_P)
- net Chainbus_addr5: now also U11.17 (GPIO11); no longer R54.1, U11.14 (GPIO8)
- net Chainbus_addr6: no longer U11.17 (GPIO11)
- new net Chainbus_addr8: R54.1, U11.14 (GPIO8)
Other:
- moved on the sheet: FB1, R43, R44, R45, R46, R47, R48

Commit message: routing done
Parts:
- added D8: TPD1E0B04DPYR, RF_TVS:X1SON-2_L1.0-W0.6-P0.65-BI, symbol RF_TVS:TPD1E0B04DPYR
Connections:
- net ANT_CN: now also D8.2
- net GND: now also D8.1
Other:
- note removed: "+Cstray"
- note removed: "ESD"
- note removed: "ESD on PSU"
- note removed: "L Value"
- note removed: "Pinout"
- note removed: "add a stub to ground pad"
- moved on the sheet: J5
Changed lines of the file:
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@@
 		)
 	)
-	(text "Pinout"
-		(exclude_from_sim no)
-		(at 259.08 175.26 0)
-		(effects
-			(font
-				(size 5.08 5.08)
-				(thickness 1.016)
-				(bold yes)
-				(color 255 0 255 1)
-			)
-		)
-	)
-	(text "ESD on PSU"
-		(exclude_from_sim no)
-		(at 158.75 96.52 0)
-		(effects
-			(font
-				(size 5.08 5.08)
-				(thickness 1.016)
-				(bold yes)
-				(color 255 0 255 1)
-			)
-		)
-	)
 	(text "USB and UART0"
 		(exclude_from_sim no)
@@
 		)
 	)
-	(text "ESD"
-		(exclude_from_sim no)
-		(at 154.94 49.53 0)
-		(effects
-			(font
-				(size 5.08 5.08)
-				(thickness 1.016)
-				(bold yes)
-				(color 255 0 255 1)
-			)
-		)
-	)
-	(text "+Cstray"
-		(exclude_from_sim no)
-		(at 81.28 191.77 0)
-		(effects
-			(font
-				(size 5.08 5.08)
-				(thickness 1.016)
-				(bold yes)
-				(color 255 0 255 1)
-			)
-		)
-	)
-	(text "add a stub\nto ground pad"
-		(exclude_from_sim no)
-		(at 48.26 50.8 0)
-		(effects
-			(font
-				(size 1.27 1.27)
-				(thickness 1.016)
-				(bold yes)
-				(color 255 0 255 1)
-			)
-		)
-	)
 	(text "Chainbus I2C"
 		(exclude_from_sim no)
@@
 		)
 	)
-	(text "L Value"
-		(exclude_from_sim no)
-		(at 67.31 154.94 0)
-		(effects
-			(font
-				(size 5.08 5.08)
-				(thickness 1.016)
-				(bold yes)
-				(color 255 0 255 1)
-			)
-		)
-	)
 	(text "SPI memory"
 		(exclude_from_sim no)
@@
 	(wire
 		(pts
-			(xy 154.94 39.37) (xy 154.94 45.72)
+			(xy 154.94 39.37) (xy 154.94 41.91)
 		)
 		(stroke
@@
 	(wire
 		(pts
-			(xy 154.94 39.37) (xy 158.75 39.37)
+			(xy 154.94 39.37) (xy 171.45 39.37)
 		)
 		(stroke
@@
 	(wire
 		(pts
-			(xy 163.83 44.45) (xy 163.83 52.07)
+			(xy 176.53 44.45) (xy 176.53 54.61)
 		)
 		(stroke
@@
 	(symbol
 		(lib_id "power:GND")
-		(at 163.83 52.07 0)
+		(at 176.53 54.61 0)
 		(mirror y)
 		(unit 1)
@@
 		(fields_autoplaced yes)
 		(property "Reference" "#PWR085"
-			(at 163.83 58.42 0)
+			(at 176.53 60.96 0)
 			(hide yes)
 			(show_name no)
@@
 		)
 		(property "Value" "GND"
-			(at 163.83 57.15 0)
+			(at 176.53 59.69 0)
 			(show_name no)
 			(do_not_autoplace no)
@@
 		)
 		(property "Footprint" ""
-			(at 163.83 52.07 0)
+			(at 176.53 54.61 0)
 			(hide yes)
 			(show_name no)
@@
 		)
 		(property "Datasheet" ""
-			(at 163.83 52.07 0)
+			(at 176.53 54.61 0)
 			(hide yes)
 			(show_name no)
@@
 		)
 		(property "Description" "Power symbol creates a global label with name \"GND\" , ground"
-			(at 163.83 52.07 0)
+			(at 176.53 54.61 0)
 			(hide yes)
 			(show_name no)
@@
 	(symbol
 		(lib_id "Connector:Conn_Coaxial")
-		(at 163.83 39.37 0)
+		(at 176.53 39.37 0)
 		(unit 1)
 		(body_style 1)
@@
 		(fields_autoplaced yes)
 		(property "Reference" "J5"
-			(at 167.64 38.3931 0)
+			(at 180.34 38.3931 0)
 			(show_name no)
 			(do_not_autoplace no)
@@
 		)
 		(property "Value" "Conn_Coaxial"
-			(at 167.64 40.9331 0)
+			(at 180.34 40.9331 0)
 			(show_name no)
 			(do_not_autoplace no)
@@
 		)
 		(property "Footprint" "Connector_Coaxial:SMA_Amphenol_901-143_Horizontal"
-			(at 163.83 39.37 0)
+			(at 176.53 39.37 0)
 			(hide yes)
 			(show_name no)
@@
 		)
 		(property "Datasheet" ""
-			(at 163.83 39.37 0)
+			(at 176.53 39.37 0)
 			(hide yes)
 			(show_name no)
@@
 		)
 		(property "Description" "coaxial connector (BNC, SMA, SMB, SMC, Cinch/RCA, LEMO, ...)"
-			(at 163.83 39.37 0)
+			(at 176.53 39.37 0)
 			(hide yes)
 			(show_name no)
@@
 					(unit 1)
 				)
+			)
+		)
+	)
+	(symbol
+		(lib_id "RF_TVS:TPD1E0B04DPYR")
+		(at 154.94 46.99 90)
+		(unit 1)
+		(body_style 1)
+		(exclude_from_sim no)
+		(in_bom yes)
+		(on_board yes)
+		(in_pos_files yes)
+		(dnp no)
+		(fields_autoplaced yes)
+		(property "Reference" "D8"
+			(at 157.48 45.7199 90)
+			(show_name no)
+			(do_not_autoplace no)
+			(effects
+				(font
+					(size 1.27 1.27)
+				)
+				(justify right)
+			)
+		)
+		(property "Value" "TPD1E0B04DPYR"
+			(at 157.48 48.2599 90)
+			(show_name no)
+			(do_not_autoplace no)
+			(effects
+				(font
+					(size 1.27 1.27)
+				)
+				(justify right)
+			)
+		)
+		(property "Footprint" "RF_TVS:X1SON-2_L1.0-W0.6-P0.65-BI"
+			(at 162.56 46.99 0)
+			(hide yes)
+			(show_name no)
+			(do_not_autoplace no)
+			(effects
+				(font
+					(size 1.27 1.27)
+				)
+			)
+		)
+		(property "Datasheet" "https://www.lcsc.com/datasheet/C1975594.pdf"
+			(at 165.1 46.99 0)
+			(hide yes)
+			(show_name no)
+			(do_not_autoplace no)
+			(effects
+				(font
+					(size 1.27 1.27)
+				)
+			)
+		)
+		(property "Description" ""
+			(at 154.94 46.99 0)
+			(hide yes)
+			(show_name no)
+			(do_not_autoplace no)
+			(effects
+				(font
+					(size 1.27 1.27)
+				)
+			)
+		)
+		(property "Manufacturer" "TI(德州仪器)"
+			(at 167.64 46.99 0)
+			(hide yes)
+			(show_name no)
+			(do_not_autoplace no)
+			(effects
+				(font
+					(size 1.27 1.27)
+				)
+			)
+		)
+		(property "MPN" "TPD1E0B04DPYR"
+			(at 170.18 46.99 0)
+			(hide yes)
+			(show_name no)
+			(do_not_autoplace no)
+			(effects
+				(font
+					(size 1.27 1.27)
+				)
+			)
+		)
+		(property "LCSC Part" "C1975594"
+			(at 172.72 46.99 0)
+			(hide yes)
+			(show_name no)
+			(do_not_autoplace no)
+			(effects
+				(font
+					(size 1.27 1.27)
+				)
+			)
+		)
+		(pin "2"
+		)
+		(pin "1"
+		)
+		(instances
+			(project "MMS3_ESP32-C6"
+				(path "/712cea22-140d-4c92-923f-f4998caf3ecd/f58b04f6-bb02-4b0f-a390-7a8ed3ac3405"
+					(reference "D8")
+					(unit 1)
+				)

Commit message: eem, done?
Parts:
- removed R50, R51: 22Ω, PCM_JLCPCB:R_0402, symbol PCM_JLCPCB-Resistors:0402,22Ω
- added R50, R51: 0Ω, PCM_JLCPCB:R_0402, symbol PCM_JLCPCB-Resistors:0402,0Ω
- J5: LCSC Part (none) -> C496551
- L3: LCSC (none) -> C2041629
Connections:
- net GPIO12: now also R50.1
- net GPIO13: now also R51.1
- net USB.D+: now also R50.2
- net USB.D-: now also R51.2
