File: MMS3/VRM.kicad_sch (KiCad schematic)
At the start: 37 parts, among them U15 AMS1117-3.3, U2 TPS54560BDDA

Commit message: finished routing
Parts:
- removed C69, C74: 100nF, PCM_JLCPCB:C_0402, symbol PCM_JLCPCB-Capacitors:0402,100nF
- added C10, C9: 100nF, PCM_JLCPCB:C_0603, symbol PCM_JLCPCB-Capacitors:0603,100nF
- C30, C31, C32, C33, C34, C35: DNP_Basic (none) -> DNP; Manufacturer Murata Electronics -> (none)
- C38, C39, C40, C41, C42, C45, C46, C47: DNP_Basic (none) -> DNP; Manufacturer Samsung Electro-Mechanics -> (none)
- C43, C44: DNP_Basic (none) -> DNP; Manufacturer FH(Guangdong Fenghua Advanced Tech) -> (none)
- C49, C50, L1, TP16, TP17, TP18, TP19, TP20, U2: DNP_Basic (none) -> DNP
- D1, D3, D4: DNP_Basic (none) -> DNP; Manufacturer hongjiacheng -> (none)
- R33, R34, R36, R37, R38, R39: DNP_Basic (none) -> DNP; Manufacturer UNI-ROYAL(Uniroyal Elec) -> (none)
Connections:
- net +3V3: now also C10.1
- net +5V: now also C9.1
- net GND: now also C10.2, C9.2
Other:
- title: MMS3 -> MMS3 MCU ESP32-C6

Commit message: eem, done?
Parts:
- TP16, TP17, TP18, TP19, TP20: now not fitted; now left out of the parts list
- U2: LCSC (none) -> C1850354

Commit message: fixed swapped RX/TX & D+/D_
Parts:
- removed R36: 43kΩ, PCM_JLCPCB:R_0603, symbol PCM_JLCPCB-Resistors:0603,43kΩ
- added C48: 22uF, PCM_JLCPCB:C_0805, symbol PCM_JLCPCB-Capacitors:0805,22uF
- added R21: 47kΩ, PCM_JLCPCB:R_0402, symbol PCM_JLCPCB-Resistors:0402,47kΩ
Connections:
- net +3V3: now also C48.1
- net GND: now also C48.2
- net Vin: no longer U2.3 (EN)
- net at C41.1, C42.1, C45.1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: now also R21.1
- net at R37.1, TP18.1, U2.5 (FB): now also R21.2
- no-connect marks 0 -> 1
Other:
- note added: "HUMAN NUMBER GENERATOR OUTPUT"
- note added: "~5.4V"
- note added: "~5V"
- moved on the sheet: D4
